File: KiCad/7segments/7segments/7segments.kicad_pcb (KiCad board)
At the start: 2 copper layers, 63.5 x 59.7 mm, 19 parts, among them J1 BC070-02-A-1-L-C_REVD1_TOP, J2 12V DC, J3 R pinnen RGB strips, SW1 ENABLE, SW2 BOOT, T1 BC848, T2 BC848, T3 BC848, T4 BC848, T5 BC848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

Commit message: kicad drawings
Parts:
- J1: value BC070-02-A-1-L-C_REVD1_TOP -> Conn_01x04_Female; footprint libraries:GCT_BC070-02-A-1-L-C_REVD1_TOP -> Connector_PinHeader_2.54mm:PinHeader_1x04_P2.54mm_Vertical
- J2: footprint libraries:TE_282841-2 -> libraries:TE_282841-3
- moved J1 6.78 mm to (170.4, 97.8), turned to 180 degrees
- moved C3 1.80 mm to (144.0, 78.7)
- moved J2 0.37 mm to (121.4, 114.5)
Connections:
- C1 pad 1: Net-(C1-Pad1) -> +3V3
- C2 pad 1: Net-(C1-Pad1) -> +3V3
- C3 pad 1: Net-(C1-Pad1) -> +3V3
- J1 pad 1: Net-(J1-Pad1) -> GND
- PS1 pad 1b: Net-(J2-Pad2) -> unconnected-(PS1-Pad1b)
- PS1 pad 2b: Net-(J2-Pad1) -> unconnected-(PS1-Pad2b)
- PS1 pad 3a: Net-(C1-Pad1) -> +3V3
- PS1 pad 3b: Net-(C1-Pad1) -> unconnected-(PS1-Pad3b)
- PS1 pad 4b: GND -> unconnected-(PS1-Pad4b)
- U1 pad 2: Net-(C1-Pad1) -> +3V3
- U1 pad 35: Net-(J1-Pad1) -> Net-(J1-Pad3)
Routing:
- net +3V3: track 0.00 -> 69.8 mm, vias 0 -> 1
- net Net-(C1-Pad1): track 34.3 -> 0.00 mm, vias 1 -> 0
- net GND: track 163.1 -> 169.7 mm
- net Net-(J2-Pad1): track 12.9 -> 6.63 mm
- net Net-(J1-Pad3): track 0.00 -> 5.57 mm
- net Net-(J1-Pad2): track 2.90 -> 6.94 mm
- net Net-(J1-Pad1): track 3.77 -> 0.00 mm
- net Net-(J3-Pad1): track 16.4 -> 15.8 mm, vias 1 -> 0
- net Net-(J3-Pad4): vias 1 -> 0
- net Net-(J3-Pad3): vias 1 -> 0
- net Net-(J3-Pad2): vias 1 -> 0
