File: KiCad/7segments/7segments/7segments.kicad_sch (KiCad schematic)
At the start: 19 parts, among them J1 BC070-02-A-1-L-C_REVD1_TOP, T2 BC848, T3 BC848, T4 BC848, T5 BC848, T6 BC848, T7 BC848, U1 ESP32-WROOM-32E_(16MB)

Commit message: kicad drawings
Parts:
- removed J1: BC070-02-A-1-L-C_REVD1_TOP, symbol BC070-02-A-1-L-C_REVD1_TOP:BC070-02-A-1-L-C_REVD1_TOP
- removed J2: (no value), symbol 282841-5:2_pin_connector
- added J1: Conn_01x04_Female, Connector_PinHeader_2.54mm:PinHeader_1x04_P2.54mm_Vertical, symbol Connector_Generic:Conn_01x04
- added J2: 12V DC, libraries:TE_282841-3, symbol 282841-3:282841-3
- C1, C2, C3: footprint (none) -> Capacitor_SMD:C_0805_2012Metric
- C4: value (none) -> 1u; footprint (none) -> Capacitor_SMD:C_0805_2012Metric
- J3: value (none) -> R pinnen RGB strips; footprint (none) -> libraries:TE_282841-8
- R1: value (none) -> 10k; footprint (none) -> libraries:RESC6332X65N
- SW1: value (none) -> ENABLE; footprint (none) -> libraries:SW_1825910-6-4
- SW2: value (none) -> BOOT; footprint (none) -> libraries:SW_1825910-6-4
- T1: value (none) -> BC848; footprint (none) -> libraries:SOT23
- T2, T3, T4, T5, T6, T7: footprint (none) -> libraries:SOT23
- U1: footprint (none) -> libraries:XCVR_ESP32-WROOM-32E_(16MB)
Connections:
- net GND: now also J1.1 (Pin_1); no longer PS1.4b (-Vout)
- net +3V3: now reaches C1.1, C2.1, C3.1, PS1.3a (+Vout), U1.2 (3V3)
- net +3V3: now also J1.4 (Pin_4); no longer PS1.3b (+Vout)
- net at U1.34 (RXD0): now also J1.2 (Pin_2)
- net at U1.35 (TXD0): now also J1.3 (Pin_3)
- net at PS1.2a (-Vin): now also J2.1; no longer PS1.2b (-Vin)
- net at PS1.1a (+Vin): now also J2.2, J2.3; no longer PS1.1b (+Vin)
- no-connect marks 17 -> 21
