File: KiCad/7segments/7segments_powerbank/7segments_powerbank.kicad_pcb (KiCad board)
At the start: 2 copper layers, 63.5 x 59.7 mm, 19 parts, among them J1 Conn_01x04_Female, J2 12V DC, J3 R pinnen RGB strips, SW1 ENABLE, SW2 BOOT, T1 BC848, T2 BC848, T3 BC848, T4 BC848, T5 BC848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

Commit message: kicad
Parts:
- R1: footprint Resistor_SMD:R_0805_2012Metric -> libraries:RESC6332X65N
- moved C3 1.30 mm to (144.0, 78.7)
- moved T2 1.02 mm to (144.0, 94.6)
Routing:
- net GND: track 196.1 -> 169.7 mm, vias 5 -> 1
- net Net-(J3-Pad7): track 34.4 -> 29.3 mm
- net +3V3: track 74.6 -> 69.8 mm
- net Net-(J3-Pad5): track 20.1 -> 17.9 mm
- net Net-(R1-Pad2): track 7.33 -> 5.19 mm
- net Net-(J3-Pad6): track 24.4 -> 22.5 mm
- net Net-(T2-Pad1): track 6.62 -> 5.40 mm
- net Net-(T4-Pad1): track 9.92 -> 9.23 mm
- net Net-(C4-Pad2): track 12.5 -> 13.0 mm
Other:
- board text removed: "7 Segment"
