File: KiCad/7segments/7segments_powerbank/7segments_powerbank.kicad_sch (KiCad schematic)
At the start: 19 parts, among them J1 Conn_01x04_Female, J2 12V DC, J3 R pinnen RGB strips, SW1 ENABLE, SW2 BOOT, T1 BC848, T2 BC848, T3 BC848, T4 BC848, T5 BC848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

Commit message: kicad
Parts:
- R1: footprint (none) -> libraries:RESC6332X65N
Changed lines of the file:
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@@
     (property "Reference" "R1" (id 0) (at 111.76 54.61 90))
     (property "Value" "10k" (id 1) (at 111.76 57.15 90))
-    (property "Footprint" "" (id 2) (at 111.76 62.738 90)
+    (property "Footprint" "libraries:RESC6332X65N" (id 2) (at 111.76 62.738 90)
       (effects (font (size 1.27 1.27)) hide)
     )
@@
     )
     (path "/079e8df5-7225-4c2f-89b7-6fc9ccc6b3d6"
-      (reference "R1") (unit 1) (value "10k") (footprint "Resistor_SMD:R_0805_2012Metric")
+      (reference "R1") (unit 1) (value "10k") (footprint "libraries:RESC6332X65N")
     )
     (path "/2e93fe94-869c-4e96-a982-fb0a32b3050b"
