File: KiCad/Buffer/Buffer/Buffer.kicad_pcb (KiCad board)
At the start: 2 copper layers, 92.7 x 61 mm, 31 parts, among them J1 Conn_01x04_Female, J2 12V DC, J3 rood, J4 oranje, J5 groen, SW1 ENABLE, SW2 BOOT, T1 signaal oranje, T10 BC848, T11 BC848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

Commit message: kicad
Parts:
- R1: footprint libraries:RESC6332X65N -> Resistor_SMD:R_0805_2012Metric
- moved C1 6.45 mm to (95.3, 79.7), turned to -90 degrees
- moved SW1 6.27 mm to (101.6, 80.0), turned to 180 degrees
- moved R1 3.64 mm to (109.2, 81.3), turned to 90 degrees
Routing:
- net Net-(R1-Pad2): track 7.68 -> 3.03 mm
- net GND: track 205.4 -> 206.2 mm
- net Net-(T3-Pad1): track 11.2 -> 11.9 mm
