File: KiCad/Buffer/Buffer/Buffer.kicad_sch (KiCad schematic)
At the start: 11 parts, among them J1 BC070-02-A-1-L-C_REVD1_TOP, SW1 ENABLE, SW2 BOOT, U1 ESP32-WROOM-32E_(16MB)

Commit message: kicad drawings
Parts:
- removed J1: BC070-02-A-1-L-C_REVD1_TOP, libraries:GCT_BC070-02-A-1-L-C_REVD1_TOP, symbol BC070-02-A-1-L-C_REVD1_TOP:BC070-02-A-1-L-C_REVD1_TOP
- removed J?: 12V DC, libraries:TE_282841-2, symbol 282841-5:2_pin_connector
- added J1: Conn_01x04_Female, Connector_PinHeader_2.54mm:PinHeader_1x04_P2.54mm_Vertical, symbol Connector_Generic:Conn_01x04
- added J2: (no value), symbol 282841-3:282841-3
- added J3: rood, libraries:TE_282841-6, symbol 282841-6:282841-6
- added J4: oranje, libraries:TE_282841-6, symbol 282841-6:282841-6
- added J5: groen, libraries:TE_282841-4, symbol 282841-5:282841-4
- added T1: signaal oranje, libraries:SOT23, symbol BC848:BC848
- added T10, T11, T12, T13, T14, T15, T16, T17, T2, T3, T4, T5, T6, T7, T8, T9: BC848, libraries:SOT23, symbol BC848:BC848
- gave numbers to parts that had none: 1
Connections:
- net GND: now also J1.1 (Pin_1), T1.2, T10.2, T11.2, T12.2, T13.2, T14.2, T15.2, T16.2, T17.2, T3.2, T5.2, T7.2, T8.2, T9.2; no longer PS1.4b (-Vout)
- net at PS1.2a (-Vin): now also J2.1; no longer PS1.2b (-Vin)
- net at PS1.1a (+Vin): now also J2.2, J2.3; no longer PS1.1b (+Vin)
- net at U1.35 (TXD0): now also J1.3 (Pin_3)
- net at U1.34 (RXD0): now also J1.2 (Pin_2)
- net at U1.10 (IO25): now also T3.1
- net at U1.11 (IO26): now also T4.1
- net at U1.12 (IO27): now also T5.1
- net at U1.13 (IO14): now also T6.1
- net at U1.14 (IO12): now also T7.1
- net at U1.16 (IO13): now also T17.1
- net +3V3: now reaches C2.1, C3.1, C4.1, PS1.3a (+Vout), U1.2 (3V3)
- net +3V3: now also J1.4 (Pin_4); no longer PS1.3b (+Vout)
- net at U1.26 (IO4): now also T15.1
- net at U1.27 (IO16): now also T13.1
- net at U1.28 (IO17): now also T11.1
- net at U1.29 (IO5): now also T16.1
- net at U1.30 (IO18): now also T14.1
- net at U1.31 (IO19): now also T12.1
- net at U1.33 (IO21): now also T10.1
- net at U1.36 (IO22): now also T9.1
- net at U1.37 (IO23): now also T8.1
- net at U1.8 (IO32): now also T1.1
- net at U1.9 (IO33): now also T2.1
- new net: T1.3, T2.2, T4.2, T6.2
- new net g1: J5.1, T17.3
- new net g2: J5.2, T15.3
- new net g3: J5.3, T13.3
- new net g4: J5.4, T11.3
- new net o1g: J4.1, T2.3
- new net o1r: J4.2, T3.3
- new net o2g: J4.3, T4.3
- new net o2r: J4.4, T5.3
- new net o3g: J4.5, T6.3
- new net o3r: J4.6, T7.3
- new net r1: J3.1, T8.3
- new net r2: J3.2, T9.3
- new net r3: J3.3, T10.3
- new net r4: J3.4, T12.3
- new net r5: J3.5, T14.3
- new net r6: J3.6, T16.3
- no-connect marks 4 -> 10
Other:
- note added: "groene lichten"
- note added: "oranje lichten - groene pulsen"
- note added: "oranje lichten - rood"
- note added: "rode lichten"

Commit message: kicad
Parts:
- J2: value (none) -> 12V DC; footprint (none) -> libraries:TE_282841-3
- R1: footprint libraries:RESC6332X65N -> (none)
Changed lines of the file:
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@@
     (property "Reference" "R1" (id 0) (at 44.45 52.07 90))
     (property "Value" "10k" (id 1) (at 44.45 54.61 90))
-    (property "Footprint" "libraries:RESC6332X65N" (id 2) (at 44.45 60.198 90)
+    (property "Footprint" "" (id 2) (at 44.45 60.198 90)
       (effects (font (size 1.27 1.27)) hide)
     )
@@
       (effects (font (size 1.27 1.27)) (justify right))
     )
-    (property "Value" "" (id 1) (at 166.37 27.9399 0)
+    (property "Value" "12V DC" (id 1) (at 166.37 27.9399 0)
       (effects (font (size 1.27 1.27)) (justify right))
     )
-    (property "Footprint" "" (id 2) (at 162.56 26.67 0)
+    (property "Footprint" "libraries:TE_282841-3" (id 2) (at 162.56 26.67 0)
       (effects (font (size 1.27 1.27)) (justify left bottom) hide)
     )
@@
     )
     (path "/0b43a8fb-b3d3-4444-a4b0-cf952c07dcfe"
-      (reference "R1") (unit 1) (value "10k") (footprint "libraries:RESC6332X65N")
+      (reference "R1") (unit 1) (value "10k") (footprint "Resistor_SMD:R_0805_2012Metric")
     )
     (path "/08ac4c42-16f0-4513-b91e-bf0b3a111257"
