File: KiCad/fiets/standaardMetVoeding (korter, beter)/standaard.kicad_sch (KiCad schematic)
At the start: 24 parts, among them J1 Conn_01x04_Female, J2 R pinnen RGB strips, J3 282837-4, J4 282841-2, J5 12V DC, SW1 ENABLE, SW2 BOOT, U1 ESP32-WROOM-32E_(16MB)

Commit message: aanpassingen
aanpass kicad fiets
Parts:
- removed J5: 12V DC, libraries:TE_282841-3, symbol 282841-3:282841-3
- added J5: 282841-2, libraries:TE_282841-2, symbol 282841-2:282841-2
- CR1, CR2, CR3, CR4: footprint Diode_SMD:D_0201_0603Metric -> Diode_SMD:D_0603_1608Metric
- R1, R2, R3, R4, R5, R6: footprint (none) -> Resistor_SMD:R_0805_2012Metric
Connections:
- net +3V3 is gone; now on an unnamed net: J1.4 (Pin_4)
- net at C2.1, C3.1, C4.1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: no longer J3.1
- net at PS1.2a (-Vin): now also J5.1
- net at PS1.1a (+Vin): now also J3.1, J5.2
