File: KiCad/standaard beginschema/standaard/standaard.kicad_sch (KiCad schematic)
At the start: 9 parts, among them J1 BC070-02-A-1-L-C_REVD1_TOP, SW1 ENABLE, SW2 BOOT, U1 ESP32-WROOM-32E_(16MB)

Commit message: update standaard kicad schema
Parts:
- removed J1: BC070-02-A-1-L-C_REVD1_TOP, libraries:GCT_BC070-02-A-1-L-C_REVD1_TOP, symbol BC070-02-A-1-L-C_REVD1_TOP:BC070-02-A-1-L-C_REVD1_TOP
- added J1: (no value), symbol Connector_Generic:Conn_01x04
Connections:
- net GND: now also J1.1 (Pin_1)
- net at U1.35 (TXD0): now also J1.3 (Pin_3)
- net at U1.34 (RXD0): now also J1.2 (Pin_2)
- net Voeding renamed +3V3
- net +3V3: now also J1.4 (Pin_4)
Changed lines of the file:
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@@
 (kicad_sch (version 20211123) (generator eeschema)
   (paper "A4")
+  (junction (at 195.58 62.23) (diameter 0) (color 0 0 0 0)
+  )
   (junction (at 88.9 86.36) (diameter 0) (color 0 0 0 0)
   )
@@
     (stroke (width 0) (type default) (color 0 0 0 0))
   )
+  (wire (pts (xy 113.03 104.14) (xy 119.38 104.14))
+    (stroke (width 0) (type default) (color 0 0 0 0))
+  )
   (wire (pts (xy 88.9 86.36) (xy 88.9 88.9))
     (stroke (width 0) (type default) (color 0 0 0 0))
@@
     (stroke (width 0) (type default) (color 0 0 0 0))
   )
-  (wire (pts (xy 196.85 62.23) (xy 185.42 62.23))
+  (wire (pts (xy 195.58 62.23) (xy 185.42 62.23))
+    (stroke (width 0) (type default) (color 0 0 0 0))
+  )
+  (wire (pts (xy 196.85 62.23) (xy 195.58 62.23))
     (stroke (width 0) (type default) (color 0 0 0 0))
   )
@@
     (stroke (width 0) (type default) (color 0 0 0 0))
   )
+  (wire (pts (xy 113.03 101.6) (xy 119.38 101.6))
+    (stroke (width 0) (type default) (color 0 0 0 0))
+  )
   (wire (pts (xy 162.56 73.66) (xy 160.02 73.66))
     (stroke (width 0) (type default) (color 0 0 0 0))
@@
     (stroke (width 0) (type default) (color 0 0 0 0))
   )
-  (global_label "Voeding" (shape input) (at 196.85 62.23 0) (fields_autoplaced)
+  (global_label "Externe Voeding" (shape input) (at 196.85 62.23 0) (fields_autoplaced)
     (effects (font (size 1.27 1.27)) (justify left))
-    (property "Intersheet References" "${INTERSHEET_REFS}" (id 0) (at 206.6412 62.1506 0)
+    (property "Intersheet References" "${INTERSHEET_REFS}" (id 0) (at 214.6241 62.1506 0)
       (effects (font (size 1.27 1.27)) (justify left) hide)
     )
@@
     (pin "1")
   )
+  (symbol (lib_id "power:+3V3") (at 195.58 62.23 0) (unit 1)
+    (in_bom yes) (on_board yes) (fields_autoplaced)
+    (property "Reference" "#PWR0109" (id 0) (at 195.58 66.04 0)
+      (effects (font (size 1.27 1.27)) hide)
+    )
+    (property "Value" "" (id 1) (at 195.58 57.15 0))
+    (property "Footprint" "" (id 2) (at 195.58 62.23 0)
+      (effects (font (size 1.27 1.27)) hide)
+    )
+    (property "Datasheet" "" (id 3) (at 195.58 62.23 0)
+      (effects (font (size 1.27 1.27)) hide)
+    )
+    (pin "1")
+  )
   (symbol (lib_id "Device:C") (at 185.42 58.42 180) (unit 1)
     (in_bom yes) (on_board yes)
@@
     (pin "4")
   )
-  (symbol (lib_id "BC070-02-A-1-L-C_REVD1_TOP:BC070-02-A-1-L-C_REVD1_TOP") (at 114.3 101.6 0) (unit 1)
-    (in_bom yes) (on_board yes) (fields_autoplaced)
-    (property "Reference" "J1" (id 0) (at 110.49 93.98 0))
-    (property "Value" "BC070-02-A-1-L-C_REVD1_TOP" (id 1) (at 110.49 96.52 0))
-    (property "Footprint" "libraries:GCT_BC070-02-A-1-L-C_REVD1_TOP" (id 2) (at 114.3 101.6 0)
-      (effects (font (size 1.27 1.27)) (justify left bottom) hide)
-    )
-    (property "Datasheet" "" (id 3) (at 114.3 101.6 0)
-      (effects (font (size 1.27 1.27)) (justify left bottom) hide)
-    )
-    (property "PARTREV" "D1" (id 4) (at 114.3 101.6 0)
-      (effects (font (size 1.27 1.27)) (justify left bottom) hide)
-    )
-    (property "MAXIMUM_PACKAGE_HEIGHT" "2.5mm" (id 5) (at 114.3 101.6 0)
-      (effects (font (size 1.27 1.27)) (justify left bottom) hide)
-    )
-    (property "MANUFACTURER" "GCT" (id 6) (at 114.3 101.6 0)
-      (effects (font (size 1.27 1.27)) (justify left bottom) hide)
-    )
-    (property "STANDARD" "Manufacturer Recommendation" (id 7) (at 114.3 101.6 0)
-      (effects (font (size 1.27 1.27)) (justify left bottom) hide)
-    )
-    (pin "1")
-    (pin "2")
+  (symbol (lib_id "power:+3V3") (at 113.03 99.06 0) (unit 1)
+    (in_bom yes) (on_board yes) (fields_autoplaced)
+    (property "Reference" "#PWR0107" (id 0) (at 113.03 102.87 0)
+      (effects (font (size 1.27 1.27)) hide)
+    )
+    (property "Value" "+3V3" (id 1) (at 113.03 93.98 0))
+    (property "Footprint" "" (id 2) (at 113.03 99.06 0)
+      (effects (font (size 1.27 1.27)) hide)
+    )
+    (property "Datasheet" "" (id 3) (at 113.03 99.06 0)
+      (effects (font (size 1.27 1.27)) hide)
+    )
+    (pin "1")
   )
   (symbol (lib_id "ESP32-WROOM-32E__16MB_:ESP32-WROOM-32E_(16MB)") (at 139.7 99.06 0) (unit 1)
@@
     (pin "9")
   )
+  (symbol (lib_id "Connector_Generic:Conn_01x04") (at 107.95 104.14 180) (unit 1)
+    (in_bom yes) (on_board yes)
+    (property "Reference" "J1" (id 0) (at 108.585 93.98 0))
+    (property "Value" "" (id 1) (at 105.41 100.33 90))
+    (property "Footprint" "" (id 2) (at 107.95 104.14 0)
+      (effects (font (size 1.27 1.27)) hide)
+    )
+    (property "Datasheet" "~" (id 3) (at 107.95 104.14 0)
+      (effects (font (size 1.27 1.27)) hide)
+    )
+    (pin "1")
+    (pin "2")
+    (pin "3")
+    (pin "4")
+  )
+  (symbol (lib_id "power:GND") (at 113.03 106.68 0) (unit 1)
+    (in_bom yes) (on_board yes)
+    (property "Reference" "#PWR0108" (id 0) (at 113.03 113.03 0)
+      (effects (font (size 1.27 1.27)) hide)
+    )
+    (property "Value" "GND" (id 1) (at 107.95 109.22 0)
+      (effects (font (size 1.27 1.27)) (justify left))
+    )
+    (property "Footprint" "" (id 2) (at 113.03 106.68 0)
+      (effects (font (size 1.27 1.27)) hide)
+    )
+    (property "Datasheet" "" (id 3) (at 113.03 106.68 0)
+      (effects (font (size 1.27 1.27)) hide)
+    )
+    (pin "1")
+  )
   (sheet_instances
     (path "/" (page "1"))
@@
       (reference "#PWR0106") (unit 1) (value "GND") (footprint "")
     )
+    (path "/c5a7322f-3853-4396-88a5-7a9f61e90230"
+      (reference "#PWR0107") (unit 1) (value "+3V3") (footprint "")
+    )
+    (path "/fbe37580-9800-44bd-928e-4503582d09e4"
+      (reference "#PWR0108") (unit 1) (value "GND") (footprint "")
+    )
+    (path "/923186cd-e689-41b9-89b8-d80614dd6061"
+      (reference "#PWR0109") (unit 1) (value "+3V3") (footprint "")
+    )
     (path "/590c7ce0-b9ae-45c9-adef-24833a8dc22d"
       (reference "C1") (unit 1) (value "1u") (footprint "Capacitor_SMD:C_0805_2012Metric")
@@
       (reference "C4") (unit 1) (value "0.1u") (footprint "Capacitor_SMD:C_0805_2012Metric")
     )
-    (path "/ceb4e362-4395-4490-bbb6-3fc3fe0af338"
-      (reference "J1") (unit 1) (value "BC070-02-A-1-L-C_REVD1_TOP") (footprint "libraries:GCT_BC070-02-A-1-L-C_REVD1_TOP")
+    (path "/ef535116-2a8d-4f09-9e81-6f8d70d5ba44"
+      (reference "J1") (unit 1) (value "Conn_01x04_Female") (footprint "Connector_PinHeader_2.54mm:PinHeader_1x04_P2.54mm_Vertical")
     )
     (path "/6d17f919-49d0-4100-b2fc-f72668e7c1f5"

Commit message: updates standaard schema
Parts:
- added R2: 10k, libraries:RESC6332X65N, symbol Device:R
- J1: value (none) -> Conn_01x04_Female; footprint (none) -> Connector_PinHeader_2.54mm:PinHeader_1x04_P2.54mm_Vertical
Connections:
- net +3V3: now also R1.1, R2.1
- net at C1.2, SW1.1, SW1.2: now also R1.2, U1.3 (EN); no longer R1.1
- net at SW2.1, SW2.2, U1.25 (IO0): now also R2.2
Other:
- moved on the sheet: C1, C2, C3, C4, R1, SW1, SW2

Commit message: kicad aanpassingen buffer
Parts:
- added J2: 12V DC, libraries:TE_282841-3, symbol 282841-3:282841-3
- added PS1: ITX0512SA, libraries:Buck Converter, symbol Converter_DCDC:ITX0512SA
Connections:
- net +3V3: now also PS1.3a (+Vout)
- net GND: now also PS1.4a (-Vout)
- new net: J2.1, PS1.2a (-Vin)
- new net: J2.2, J2.3, PS1.1a (+Vin)
- no-connect marks 16 -> 20
Changed lines of the file:
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@@
 (kicad_sch (version 20211123) (generator eeschema)
   (paper "A4")
-  (junction (at 195.58 58.42) (diameter 0) (color 0 0 0 0)
-  )
   (junction (at 93.98 86.36) (diameter 0) (color 0 0 0 0)
   )
@@
   (junction (at 93.98 78.74) (diameter 0) (color 0 0 0 0)
   )
+  (junction (at 199.39 58.42) (diameter 0) (color 0 0 0 0)
+  )
+  (junction (at 229.87 53.34) (diameter 0) (color 0 0 0 0)
+  )
   (junction (at 165.1 58.42) (diameter 0) (color 0 0 0 0)
   )
@@
   (junction (at 175.26 58.42) (diameter 0) (color 0 0 0 0)
   )
+  (no_connect (at 226.06 48.26))
   (no_connect (at 119.38 93.98))
   (no_connect (at 160.02 104.14))
@@
   (no_connect (at 119.38 91.44))
   (no_connect (at 119.38 81.28))
+  (no_connect (at 205.74 48.26))
   (no_connect (at 160.02 99.06))
+  (no_connect (at 226.06 55.88))
   (no_connect (at 160.02 96.52))
   (no_connect (at 160.02 78.74))
   (no_connect (at 160.02 106.68))
+  (no_connect (at 205.74 55.88))
   (no_connect (at 160.02 81.28))
   (no_connect (at 160.02 101.6))
@@
     (stroke (width 0) (type default) (color 0 0 0 0))
   )
+  (wire (pts (xy 226.06 50.8) (xy 229.87 50.8))
+    (stroke (width 0) (type default) (color 0 0 0 0))
+  )
   (wire (pts (xy 93.98 86.36) (xy 93.98 88.9))
     (stroke (width 0) (type default) (color 0 0 0 0))
@@
     (stroke (width 0) (type default) (color 0 0 0 0))
   )
-  (wire (pts (xy 195.58 58.42) (xy 185.42 58.42))
-    (stroke (width 0) (type default) (color 0 0 0 0))
-  )
-  (wire (pts (xy 196.85 58.42) (xy 195.58 58.42))
+  (wire (pts (xy 205.74 58.42) (xy 199.39 58.42))
+    (stroke (width 0) (type default) (color 0 0 0 0))
+  )
+  (wire (pts (xy 185.42 58.42) (xy 199.39 58.42))
     (stroke (width 0) (type default) (color 0 0 0 0))
   )
@@
     (stroke (width 0) (type default) (color 0 0 0 0))
   )
+  (wire (pts (xy 226.06 58.42) (xy 227.33 58.42))
+    (stroke (width 0) (type default) (color 0 0 0 0))
+  )
+  (wire (pts (xy 227.33 53.34) (xy 229.87 53.34))
+    (stroke (width 0) (type default) (color 0 0 0 0))
+  )
   (wire (pts (xy 93.98 78.74) (xy 93.98 86.36))
     (stroke (width 0) (type default) (color 0 0 0 0))
@@
     (stroke (width 0) (type default) (color 0 0 0 0))
   )
+  (wire (pts (xy 229.87 53.34) (xy 229.87 55.88))
+    (stroke (width 0) (type default) (color 0 0 0 0))
+  )
   (wire (pts (xy 116.84 73.66) (xy 119.38 73.66))
     (stroke (width 0) (type default) (color 0 0 0 0))
@@
     (stroke (width 0) (type default) (color 0 0 0 0))
   )
-  (global_label "Externe Voeding" (shape input) (at 196.85 58.42 0) (fields_autoplaced)
-    (effects (font (size 1.27 1.27)) (justify left))
-    (property "Intersheet References" "${INTERSHEET_REFS}" (id 0) (at 214.6241 58.3406 0)
-      (effects (font (size 1.27 1.27)) (justify left) hide)
-    )
+  (wire (pts (xy 227.33 58.42) (xy 227.33 53.34))
+    (stroke (width 0) (type default) (color 0 0 0 0))
   )
   (symbol (lib_id "power:GND") (at 160.02 127 0) (unit 1)
@@
     (pin "1")
     (pin "2")
+  )
+  (symbol (lib_id "282841-3:282841-3") (at 240.03 53.34 0) (mirror y) (unit 1)
+    (in_bom yes) (on_board yes) (fields_autoplaced)
+    (property "Reference" "J2" (id 0) (at 243.84 52.0699 0)
+      (effects (font (size 1.27 1.27)) (justify right))
+    )
+    (property "Value" "12V DC" (id 1) (at 243.84 54.6099 0)
+      (effects (font (size 1.27 1.27)) (justify right))
+    )
+    (property "Footprint" "libraries:TE_282841-3" (id 2) (at 240.03 53.34 0)
+      (effects (font (size 1.27 1.27)) (justify left bottom) hide)
+    )
+    (property "Datasheet" "" (id 3) (at 240.03 53.34 0)
+      (effects (font (size 1.27 1.27)) (justify left bottom) hide)
+    )
+    (property "Comment" "282841-3" (id 4) (at 240.03 53.34 0)
+      (effects (font (size 1.27 1.27)) (justify left bottom) hide)
+    )
+    (property "EU_RoHS_Compliance" "Compliant with Exemptions" (id 5) (at 240.03 53.34 0)
+      (effects (font (size 1.27 1.27)) (justify left bottom) hide)
+    )
+    (pin "1")
+    (pin "2")
+    (pin "3")
   )
   (symbol (lib_id "power:+3V3") (at 116.84 66.04 0) (unit 1)
@@
     (pin "2")
   )
-  (symbol (lib_id "power:+3V3") (at 195.58 58.42 0) (unit 1)
-    (in_bom yes) (on_board yes) (fields_autoplaced)
-    (property "Reference" "#PWR0109" (id 0) (at 195.58 62.23 0)
-      (effects (font (size 1.27 1.27)) hide)
-    )
-    (property "Value" "+3V3" (id 1) (at 195.58 53.34 0))
-    (property "Footprint" "" (id 2) (at 195.58 58.42 0)
-      (effects (font (size 1.27 1.27)) hide)
-    )
-    (property "Datasheet" "" (id 3) (at 195.58 58.42 0)
+  (symbol (lib_id "power:GND") (at 205.74 50.8 270) (unit 1)
+    (in_bom yes) (on_board yes)
+    (property "Reference" "#PWR0112" (id 0) (at 199.39 50.8 0)
+      (effects (font (size 1.27 1.27)) hide)
+    )
+    (property "Value" "GND" (id 1) (at 201.93 48.26 90)
+      (effects (font (size 1.27 1.27)) (justify left))
+    )
+    (property "Footprint" "" (id 2) (at 205.74 50.8 0)
+      (effects (font (size 1.27 1.27)) hide)
+    )
+    (property "Datasheet" "" (id 3) (at 205.74 50.8 0)
+      (effects (font (size 1.27 1.27)) hide)
+    )
+    (pin "1")
+  )
+  (symbol (lib_id "power:+3V3") (at 199.39 58.42 0) (unit 1)
+    (in_bom yes) (on_board yes) (fields_autoplaced)
+    (property "Reference" "#PWR0109" (id 0) (at 199.39 62.23 0)
+      (effects (font (size 1.27 1.27)) hide)
+    )
+    (property "Value" "+3V3" (id 1) (at 199.39 53.34 0))
+    (property "Footprint" "" (id 2) (at 199.39 58.42 0)
+      (effects (font (size 1.27 1.27)) hide)
+    )
+    (property "Datasheet" "" (id 3) (at 199.39 58.42 0)
       (effects (font (size 1.27 1.27)) hide)
     )
@@
     (pin "3")
     (pin "4")
+  )
+  (symbol (lib_id "Converter_DCDC:ITX0512SA") (at 215.9 53.34 180) (unit 1)
+    (in_bom yes) (on_board yes)
+    (property "Reference" "PS1" (id 0) (at 215.9 41.91 0))
+    (property "Value" "ITX0512SA" (id 1) (at 215.9 44.45 0))
+    (property "Footprint" "libraries:Buck Converter" (id 2) (at 242.57 46.99 0)
+      (effects (font (size 1.27 1.27)) (justify left) hide)
+    )
+    (property "Datasheet" "" (id 3) (at 189.23 45.72 0)
+      (effects (font (size 1.27 1.27)) (justify left) hide)
+    )
+    (pin "1a")
+    (pin "1b")
+    (pin "2a")
+    (pin "2b")
+    (pin "3a")
+    (pin "3b")
+    (pin "4a")
+    (pin "4b")
   )
   (symbol (lib_id "power:+3V3") (at 165.1 66.04 0) (unit 1)
@@
       (reference "#PWR0111") (unit 1) (value "+3V3") (footprint "")
     )
+    (path "/8f8bb641-6f96-48dd-a2de-b7e2aaf6efe0"
+      (reference "#PWR0112") (unit 1) (value "GND") (footprint "")
+    )
     (path "/590c7ce0-b9ae-45c9-adef-24833a8dc22d"
       (reference "C1") (unit 1) (value "1u") (footprint "Capacitor_SMD:C_0805_2012Metric")
@@
       (reference "J1") (unit 1) (value "Conn_01x04_Female") (footprint "Connector_PinHeader_2.54mm:PinHeader_1x04_P2.54mm_Vertical")
     )
+    (path "/52d326d4-51c9-4c17-8412-9aaf3e6cdf4c"
+      (reference "J2") (unit 1) (value "12V DC") (footprint "libraries:TE_282841-3")
+    )
+    (path "/ac81fb15-6f1a-451b-a962-fb87ffd26f6b"
+      (reference "PS1") (unit 1) (value "ITX0512SA") (footprint "libraries:Buck Converter")
+    )
     (path "/6d17f919-49d0-4100-b2fc-f72668e7c1f5"
