File: KiCad/7segments/7segments - versie met convertor/7segments.kicad_pcb (KiCad board)
At the start: 2 copper layers, 63.5 x 59.7 mm, 24 parts, among them J1 Conn_01x04_Female, J3 R pinnen RGB strips, SW1 ENABLE, SW2 BOOT, T1 BC848, T2 BC848, T3 BC848, T4 BC848, T5 BC848, T6 BC848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

Commit message: aanpass kicad
Routing:
- added copper zone on B.Cu, net GND
- added copper zone on F.Cu, net GND
Changed lines of the file:
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@@
   (segment (start 166.23 102.69) (end 166.23 103.58) (width 0.7) (layer "F.Cu") (net 45))
   (segment (start 170.398 113.74) (end 170.398 107.24) (width 0.7) (layer "B.Cu") (net 45))
+  (zone (net 2) (net_name "GND") (layers F&B.Cu) (hatch edge 0.508)
+    (connect_pads (clearance 0.508))
+    (min_thickness 0.254) (filled_areas_thickness no)
+    (fill yes (thermal_gap 0.508) (thermal_bridge_width 0.508))
+    (polygon
+      (pts
+        (xy 175.895 130.429)
+        (xy 113.665 130.048)
+        (xy 113.284 71.755)
+        (xy 175.514 71.755)
+      )
+    )
+  )
 )
