File: KiCad/7segments/7segments - versie met convertor/7segments.kicad_sch (KiCad schematic)
At the start: 25 parts, among them J1 Conn_01x04_Female, J3 R pinnen RGB strips, SW1 ENABLE, SW2 BOOT, T1 BC848, T2 BC848, T3 BC848, T4 BC848, T5 BC848, T6 BC848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

Commit message: aanpass kicad
Parts:
- removed J2: (no value), symbol Connector:Conn_01x01_Male
Connections:
- net at J3.8: now also PS1.1a (+Vin)
Other:
- note removed: "Naar 12V ledstrips"
- note removed: "welk soort connector???"
Changed lines of the file:
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@@
   (junction (at 162.56 46.99) (diameter 0) (color 0 0 0 0)
   )
-  (junction (at 231.14 63.5) (diameter 0) (color 0 0 0 0)
-  )
   (junction (at 199.39 63.5) (diameter 0) (color 0 0 0 0)
   )
@@
   )
   (junction (at 128.27 83.82) (diameter 0) (color 0 0 0 0)
+  )
+  (junction (at 229.87 63.5) (diameter 0) (color 0 0 0 0)
   )
   (junction (at 171.45 46.99) (diameter 0) (color 0 0 0 0)
@@
   (no_connect (at 234.95 55.88))
   (no_connect (at 207.01 60.96))
-  (no_connect (at 182.88 124.46))
+  (no_connect (at 241.3 125.73))
   (no_connect (at 77.47 109.22))
   (no_connect (at 77.47 111.76))
@@
   (no_connect (at 118.11 99.06))
   (no_connect (at 118.11 93.98))
-  (polyline (pts (xy 256.54 76.2) (xy 228.6 76.2))
-    (stroke (width 0) (type default) (color 0 0 0 0))
-  )
   (wire (pts (xy 175.26 137.16) (xy 175.26 114.3))
     (stroke (width 0) (type default) (color 0 0 0 0))
@@
     (stroke (width 0) (type default) (color 0 0 0 0))
   )
-  (polyline (pts (xy 228.6 66.04) (xy 256.54 66.04))
-    (stroke (width 0) (type default) (color 0 0 0 0))
-  )
   (wire (pts (xy 123.19 63.5) (xy 133.35 63.5))
     (stroke (width 0) (type default) (color 0 0 0 0))
@@
     (stroke (width 0) (type default) (color 0 0 0 0))
   )
+  (wire (pts (xy 229.87 63.5) (xy 234.95 63.5))
+    (stroke (width 0) (type default) (color 0 0 0 0))
+  )
   (wire (pts (xy 138.43 120.65) (xy 138.43 124.46))
     (stroke (width 0) (type default) (color 0 0 0 0))
@@
     (stroke (width 0) (type default) (color 0 0 0 0))
   )
+  (wire (pts (xy 182.88 130.81) (xy 182.88 124.46))
+    (stroke (width 0) (type default) (color 0 0 0 0))
+  )
   (wire (pts (xy 173.99 129.54) (xy 173.99 142.24))
     (stroke (width 0) (type default) (color 0 0 0 0))
@@
     (stroke (width 0) (type default) (color 0 0 0 0))
   )
-  (wire (pts (xy 231.14 63.5) (xy 234.95 63.5))
+  (wire (pts (xy 227.33 63.5) (xy 229.87 63.5))
     (stroke (width 0) (type default) (color 0 0 0 0))
   )
@@
     (stroke (width 0) (type default) (color 0 0 0 0))
   )
-  (wire (pts (xy 227.33 63.5) (xy 231.14 63.5))
-    (stroke (width 0) (type default) (color 0 0 0 0))
-  )
   (wire (pts (xy 128.27 106.68) (xy 128.27 119.38))
     (stroke (width 0) (type default) (color 0 0 0 0))
@@
     (stroke (width 0) (type default) (color 0 0 0 0))
   )
-  (polyline (pts (xy 256.54 66.04) (xy 256.54 76.2))
-    (stroke (width 0) (type default) (color 0 0 0 0))
-  )
   (wire (pts (xy 138.43 143.51) (xy 138.43 147.32))
     (stroke (width 0) (type default) (color 0 0 0 0))
@@
     (stroke (width 0) (type default) (color 0 0 0 0))
   )
+  (wire (pts (xy 229.87 130.81) (xy 182.88 130.81))
+    (stroke (width 0) (type default) (color 0 0 0 0))
+  )
   (wire (pts (xy 162.56 46.99) (xy 158.75 46.99))
     (stroke (width 0) (type default) (color 0 0 0 0))
@@
     (stroke (width 0) (type default) (color 0 0 0 0))
   )
+  (wire (pts (xy 229.87 63.5) (xy 229.87 130.81))
+    (stroke (width 0) (type default) (color 0 0 0 0))
+  )
   (wire (pts (xy 118.11 134.62) (xy 143.51 134.62))
     (stroke (width 0) (type default) (color 0 0 0 0))
@@
   )
   (wire (pts (xy 72.39 91.44) (xy 77.47 91.44))
-    (stroke (width 0) (type default) (color 0 0 0 0))
-  )
-  (polyline (pts (xy 228.6 66.04) (xy 228.6 76.2))
     (stroke (width 0) (type default) (color 0 0 0 0))
   )
@@
   (text "Hieraan hangen we onze\nDC-DC convertor \n(gevoed met een powerbank, 5V)"
     (at 241.3 62.23 0)
-    (effects (font (size 1.27 1.27)) (justify left bottom))
-  )
-  (text "welk soort connector???" (at 229.87 78.74 0)
-    (effects (font (size 1.27 1.27)) (justify left bottom))
-  )
-  (text "Naar 12V ledstrips\n" (at 232.41 73.66 0)
     (effects (font (size 1.27 1.27)) (justify left bottom))
   )
@@
     (pin "2")
   )
-  (symbol (lib_id "Connector:Conn_01x01_Male") (at 231.14 68.58 90) (unit 1)
-    (in_bom yes) (on_board yes) (fields_autoplaced)
-    (property "Reference" "J2" (id 0) (at 232.41 66.6749 90)
-      (effects (font (size 1.27 1.27)) (justify right))
-    )
-    (property "Value" "" (id 1) (at 232.41 69.2149 90)
-      (effects (font (size 1.27 1.27)) (justify right))
-    )
-    (property "Footprint" "" (id 2) (at 231.14 68.58 0)
-      (effects (font (size 1.27 1.27)) hide)
-    )
-    (property "Datasheet" "~" (id 3) (at 231.14 68.58 0)
-      (effects (font (size 1.27 1.27)) hide)
-    )
-    (pin "1")
-  )
   (symbol (lib_id "1825910-6:1825910-6") (at 59.69 93.98 180) (unit 1)
     (in_bom yes) (on_board yes) (fields_autoplaced)
@@
       (reference "J1") (unit 1) (value "Conn_01x04_Female") (footprint "Connector_PinHeader_2.54mm:PinHeader_1x04_P2.54mm_Vertical")
     )
-    (path "/f99577ed-73e8-41c0-ae19-e9b3555676c3"
-      (reference "J2") (unit 1) (value "Conn_01x01_Male") (footprint "Connector_PinHeader_2.54mm:PinHeader_1x01_P2.54mm_Vertical")
-    )
     (path "/1842b158-5de9-40ef-b815-cc6428c97c75"
