File: KiCad/7segments/7segment/7segment.kicad_sch (KiCad schematic)
At the start: 20 parts, among them J1 Conn_01x04_Female, J2 12V DC, J3 R pinnen RGB strips, SW1 ENABLE, SW2 BOOT, T1 BC848, T2 BC848, T3 BC848, T4 BC848, T5 BC848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

Commit message: updaten van 7 segment ground plane(s)
versie voor 7 segment met 1 ground plane aan achterkant en andere versie met ground plane aan voor- en achterkant
Parts:
- removed J2: 12V DC, libraries:TE_282841-3, symbol 282841-3:282841-3
- added C5, C7: 0.1u, Capacitor_SMD:C_0805_2012Metric, symbol Device:C
- added C6, C8: 4.7u, Capacitor_SMD:C_0805_2012Metric, symbol Device:C
- added J2: 12V DC, libraries:TE_282841-2, symbol 282841-2:282841-2
- added U2: AMS1117, libraries:SOT229P700X180-4N, symbol AMS1117:AMS1117
Connections:
- net +3V3: now also C5.1, C6.1, U2.2 (VOUT), U2.4 (VOUT); no longer PS1.3a (+Vout)
- net GND: now also PS1.2a (-Vin), C5.2, C6.2, C7.1, C8.2, J2.2, U2.1 (ADJ/GND)
- net 12V: now reaches J3.8
- net 12V: now also PS1.1a (+Vin), J2.1
- new net: C7.2, C8.1, PS1.3a (+Vout), U2.3 (VIN)
- no-connect marks 21 -> 20
Other:
- note removed: "Hier misschien nog een component insteken waar we de laptopadapter rechtstreeks in kunnen steken"
- moved on the sheet: C1, C2, C3, C4, J1, J3, PS1, R1, R2, SW1, SW2, T1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
