File: KiCad/7segments/7segments_achterkant_groundplane/7segments.kicad_pcb (KiCad board)
At the start: 2 copper layers, 72.4 x 55.9 mm, 25 parts, among them J1 Conn_01x04_Female, J2 12V DC, J3 R pinnen RGB strips, SW1 ENABLE, SW2 BOOT, T1 BC848, T2 BC848, T3 BC848, T4 BC848, T5 BC848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

Commit message: aanpassingen aan kicad ontwerpen van 7segment en buffer
toevoeging van groundplanes
Parts:
- C1: footprint Capacitor_SMD:C_0805_2012Metric -> libraries:CAP_EEE0JA101WR
- J2: footprint libraries:TE_282841-3 -> libraries:TE_282841-2
- moved U2 2.50 mm to (122.6, 78.4)
- moved J2 2.44 mm to (113.1, 82.4), turned to 90 degrees
- moved C1 1.58 mm to (130.3, 78.2)
- moved C2 0.35 mm to (134.8, 79.1)
Connections:
- J2 pad 1: GND -> 12V
- J2 pad 2: Net-(J2-Pad2) -> GND
- J3 pad 8: unconnected-(J3-Pad8) -> 12V
- PS1 pad 1a: Net-(J2-Pad2) -> 12V
Routing:
- net 12V: track 0.00 -> 46.3 mm
- net Net-(J2-Pad2): track 27.0 -> 0.00 mm
- net +3V3: track 91.7 -> 94.4 mm
- net GND: track 97.1 -> 99.6 mm
- net Net-(C7-Pad2): track 28.9 -> 29.7 mm
