File: KiCad/7segments/7segments_beide_groundplane/7segments_beide_groundplane.kicad_pcb (KiCad board)
At the start: 2 copper layers, 72.4 x 55.9 mm, 25 parts, among them J1 Conn_01x04_Female, J2 12V DC, J3 R pinnen RGB strips, SW1 ENABLE, SW2 BOOT, T1 BC848, T2 BC848, T3 BC848, T4 BC848, T5 BC848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

Commit message: cut-outs groundplanes onder antenne
enkel voor 7 segments en buffer
Routing:
- net GND: vias 3 -> 7
Changed lines of the file:
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@@
   (segment (start 146.05 84.248598) (end 146.05 86.36) (width 0.8) (layer "F.Cu") (net 1))
   (segment (start 137.3 80.05) (end 140.1 80.05) (width 0.8) (layer "F.Cu") (net 1))
+  (via (at 113.9 116) (size 1.5) (drill 0.8) (layers "F.Cu" "B.Cu") (free) (net 2))
   (via (at 144.9 103.4) (size 1.5) (drill 0.8) (layers "F.Cu" "B.Cu") (free) (net 2))
   (via (at 140.1 96.8) (size 1.5) (drill 0.8) (layers "F.Cu" "B.Cu") (free) (net 2))
   (via (at 141.2 101.9) (size 1.5) (drill 0.8) (layers "F.Cu" "B.Cu") (free) (net 2))
+  (via (at 166.4 72.7) (size 1.5) (drill 0.8) (layers "F.Cu" "B.Cu") (free) (net 2))
+  (via (at 115 73.1) (size 1.5) (drill 0.8) (layers "F.Cu" "B.Cu") (free) (net 2))
+  (via (at 168.2 118.5) (size 1.5) (drill 0.8) (layers "F.Cu" "B.Cu") (free) (net 2))
   (segment (start 158 114.78) (end 158 108) (width 0.8) (layer "F.Cu") (net 3))
   (segment (start 156.98 115.8) (end 158 114.78) (width 0.8) (layer "F.Cu") (net 3))
@@
       )
     )
+    (polygon
+      (pts
+        (xy 147.35 77.5)
+        (xy 147.35 85.55)
+        (xy 167.6 85.55)
+        (xy 167.6 77.5)
+      )
+    )
