File: KiCad/7segments/7segments_beide_groundplane/7segments_beide_groundplane.kicad_pcb (KiCad board)
At the start: 2 copper layers, 72.4 x 55.9 mm, 25 parts, among them J1 Conn_01x04_Female, J2 12V DC, J3 R pinnen RGB strips, SW1 ENABLE, SW2 BOOT, T1 BC848, T2 BC848, T3 BC848, T4 BC848, T5 BC848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

Commit message: updates kroonsteentjes naar 2.54mm voor 7segment en buffer
Parts:
- J3: footprint libraries:TE_282841-8 -> libraries:TE_1546215-8
- T1, T2, T3, T4, T5, T6, T7: value BC848 -> NTR4503
- moved PS1 3.02 mm to (119.2, 101.5)
- moved J3 2.45 mm to (141.6, 116.3)
- moved J1 0.40 mm to (170.3, 95.2)
Routing:
- net 12V: track 42.1 -> 51.7 mm
- net Net-(J3-Pad1): track 8.22 -> 12.4 mm
- net +3V3: track 93.2 -> 95.9 mm
- net Net-(J3-Pad2): track 7.17 -> 8.98 mm
- net Net-(C7-Pad2): track 28.5 -> 30.3 mm
- net Net-(J3-Pad4): track 9.37 -> 10.2 mm

Commit message: aanmaak mapje voor finale ontwerpen
Routing:
- net GND: vias 7 -> 9
Changed lines of the file:
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@@
   (segment (start 137.3 80.05) (end 140.1 80.05) (width 0.8) (layer "F.Cu") (net 1))
   (via (at 113.9 116) (size 1.5) (drill 0.8) (layers "F.Cu" "B.Cu") (free) (net 2))
+  (via (at 142.2 91.2) (size 1.5) (drill 0.8) (layers "F.Cu" "B.Cu") (free) (net 2))
   (via (at 144.9 103.4) (size 1.5) (drill 0.8) (layers "F.Cu" "B.Cu") (free) (net 2))
   (via (at 140.1 96.8) (size 1.5) (drill 0.8) (layers "F.Cu" "B.Cu") (free) (net 2))
+  (via (at 147.6 111.6) (size 1.5) (drill 0.8) (layers "F.Cu" "B.Cu") (free) (net 2))
   (via (at 141.2 101.9) (size 1.5) (drill 0.8) (layers "F.Cu" "B.Cu") (free) (net 2))
   (via (at 166.4 72.7) (size 1.5) (drill 0.8) (layers "F.Cu" "B.Cu") (free) (net 2))
