File: KiCad/7segments/7segments_beide_groundplane/7segments_beide_groundplane.kicad_sch (KiCad schematic)
At the start: 25 parts, among them J1 Conn_01x04_Female, J2 12V DC, J3 R pinnen RGB strips, SW1 ENABLE, SW2 BOOT, T1 BC848, T2 BC848, T3 BC848, T4 BC848, T5 BC848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

Commit message: aanpassingen aan kicad ontwerpen van 7segment en buffer
toevoeging van groundplanes
Parts:
- C1: footprint Capacitor_SMD:C_0805_2012Metric -> (none)
- J2: footprint (none) -> libraries:TE_282841-2
Changed lines of the file:
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@@
     (property "Reference" "J2" (id 0) (at 234.95 40.64 0))
     (property "Value" "12V DC" (id 1) (at 234.95 43.18 0))
-    (property "Footprint" "" (id 2) (at 236.22 48.26 0)
+    (property "Footprint" "libraries:TE_282841-2" (id 2) (at 236.22 48.26 0)
       (effects (font (size 1.27 1.27)) (justify left bottom) hide)
     )
@@
       (effects (font (size 1.27 1.27)) (justify right))
     )
-    (property "Footprint" "Capacitor_SMD:C_0805_2012Metric" (id 2) (at 105.7148 48.26 0)
+    (property "Footprint" "" (id 2) (at 105.7148 48.26 0)
       (effects (font (size 1.27 1.27)) hide)
     )
@@
     )
     (path "/ca3bfd12-a47a-49d0-a984-db6af30b3c2f"
-      (reference "C1") (unit 1) (value "220u") (footprint "Capacitor_SMD:C_0805_2012Metric")
+      (reference "C1") (unit 1) (value "220u") (footprint "libraries:CAP_EEE0JA101WR")
     )
     (path "/4f6e295a-eda9-488f-8a54-b432f357af54"

Commit message: cut-outs groundplanes onder antenne
enkel voor 7 segments en buffer
Parts:
- C1: footprint (none) -> libraries:CAP_EEE0JA101WR
- T1: value BC848 -> (none); footprint libraries:SOT23 -> (none)
- T2, T3, T4, T5, T6, T7: value BC848 -> (none)
Changed lines of the file:
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@@
     (in_bom yes) (on_board yes) (fields_autoplaced)
     (property "Reference" "T1" (id 0) (at 111.76 119.38 90))
-    (property "Value" "BC848" (id 1) (at 111.76 121.92 90))
-    (property "Footprint" "libraries:SOT23" (id 2) (at 111.76 114.3 0)
+    (property "Value" "" (id 1) (at 111.76 121.92 90))
+    (property "Footprint" "" (id 2) (at 111.76 114.3 0)
       (effects (font (size 1.27 1.27)) (justify left bottom) hide)
     )
@@
     (in_bom yes) (on_board yes) (fields_autoplaced)
     (property "Reference" "T6" (id 0) (at 142.24 142.24 90))
-    (property "Value" "BC848" (id 1) (at 142.24 144.78 90))
+    (property "Value" "" (id 1) (at 142.24 144.78 90))
     (property "Footprint" "libraries:SOT23" (id 2) (at 142.24 137.16 0)
       (effects (font (size 1.27 1.27)) (justify left bottom) hide)
@@
     (in_bom yes) (on_board yes) (fields_autoplaced)
     (property "Reference" "T4" (id 0) (at 127 142.24 90))
-    (property "Value" "BC848" (id 1) (at 127 144.78 90))
+    (property "Value" "" (id 1) (at 127 144.78 90))
     (property "Footprint" "libraries:SOT23" (id 2) (at 127 137.16 0)
       (effects (font (size 1.27 1.27)) (justify left bottom) hide)
@@
     (in_bom yes) (on_board yes) (fields_autoplaced)
     (property "Reference" "T5" (id 0) (at 142.24 119.38 90))
-    (property "Value" "BC848" (id 1) (at 142.24 121.92 90))
+    (property "Value" "" (id 1) (at 142.24 121.92 90))
     (property "Footprint" "libraries:SOT23" (id 2) (at 142.24 114.3 0)
       (effects (font (size 1.27 1.27)) (justify left bottom) hide)
@@
     (in_bom yes) (on_board yes) (fields_autoplaced)
     (property "Reference" "T7" (id 0) (at 157.48 142.24 90))
-    (property "Value" "BC848" (id 1) (at 157.48 144.78 90))
+    (property "Value" "" (id 1) (at 157.48 144.78 90))
     (property "Footprint" "libraries:SOT23" (id 2) (at 157.48 137.16 0)
       (effects (font (size 1.27 1.27)) (justify left bottom) hide)
@@
     (in_bom yes) (on_board yes) (fields_autoplaced)
     (property "Reference" "T2" (id 0) (at 111.76 142.24 90))
-    (property "Value" "BC848" (id 1) (at 111.76 144.78 90))
+    (property "Value" "" (id 1) (at 111.76 144.78 90))
     (property "Footprint" "libraries:SOT23" (id 2) (at 111.76 137.16 0)
       (effects (font (size 1.27 1.27)) (justify left bottom) hide)
@@
       (effects (font (size 1.27 1.27)) (justify right))
     )
-    (property "Footprint" "" (id 2) (at 105.7148 48.26 0)
+    (property "Footprint" "libraries:CAP_EEE0JA101WR" (id 2) (at 105.7148 48.26 0)
       (effects (font (size 1.27 1.27)) hide)
     )
@@
     (in_bom yes) (on_board yes) (fields_autoplaced)
     (property "Reference" "T3" (id 0) (at 127 119.38 90))
-    (property "Value" "BC848" (id 1) (at 127 121.92 90))
+    (property "Value" "" (id 1) (at 127 121.92 90))
     (property "Footprint" "libraries:SOT23" (id 2) (at 127 114.3 0)
       (effects (font (size 1.27 1.27)) (justify left bottom) hide)
@@
     )
     (path "/0b1ac98c-8e00-4f58-bcdc-36a12707f048"
-      (reference "T1") (unit 1) (value "BC848") (footprint "libraries:SOT23")
+      (reference "T1") (unit 1) (value "NTR4503") (footprint "libraries:SOT23")
     )
     (path "/c84ee2ff-79df-4e24-aa42-638b2c557dbb"
-      (reference "T2") (unit 1) (value "BC848") (footprint "libraries:SOT23")
+      (reference "T2") (unit 1) (value "NTR4503") (footprint "libraries:SOT23")
     )
     (path "/e3e6331e-58ed-4b21-b723-09d3895539b6"
-      (reference "T3") (unit 1) (value "BC848") (footprint "libraries:SOT23")
+      (reference "T3") (unit 1) (value "NTR4503") (footprint "libraries:SOT23")
     )
     (path "/8ebe6344-8c02-465e-b9bd-92a15575c6c1"
-      (reference "T4") (unit 1) (value "BC848") (footprint "libraries:SOT23")
+      (reference "T4") (unit 1) (value "NTR4503") (footprint "libraries:SOT23")
     )
     (path "/9be3a68e-fcc2-4c4b-9ac3-35e8c8a13fe2"
-      (reference "T5") (unit 1) (value "BC848") (footprint "libraries:SOT23")
+      (reference "T5") (unit 1) (value "NTR4503") (footprint "libraries:SOT23")
     )
     (path "/3f086888-77a8-4b41-a407-5084a469d26b"
-      (reference "T6") (unit 1) (value "BC848") (footprint "libraries:SOT23")
+      (reference "T6") (unit 1) (value "NTR4503") (footprint "libraries:SOT23")
     )
     (path "/b0ff528e-2887-4136-b427-576c0ce94faf"
-      (reference "T7") (unit 1) (value "BC848") (footprint "libraries:SOT23")
+      (reference "T7") (unit 1) (value "NTR4503") (footprint "libraries:SOT23")
     )
     (path "/20bfcf3a-9cde-4c7f-a967-40b16ec717fd"

Commit message: kicad fiets hertekend
Parts:
- T1: value (none) -> NTR4503; footprint (none) -> libraries:SOT23
- T2, T3, T4, T5, T6, T7: value (none) -> NTR4503
Changed lines of the file:
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@@
     (in_bom yes) (on_board yes) (fields_autoplaced)
     (property "Reference" "T1" (id 0) (at 111.76 119.38 90))
-    (property "Value" "" (id 1) (at 111.76 121.92 90))
-    (property "Footprint" "" (id 2) (at 111.76 114.3 0)
+    (property "Value" "NTR4503" (id 1) (at 111.76 121.92 90))
+    (property "Footprint" "libraries:SOT23" (id 2) (at 111.76 114.3 0)
       (effects (font (size 1.27 1.27)) (justify left bottom) hide)
     )
@@
     (in_bom yes) (on_board yes) (fields_autoplaced)
     (property "Reference" "T6" (id 0) (at 142.24 142.24 90))
-    (property "Value" "" (id 1) (at 142.24 144.78 90))
+    (property "Value" "NTR4503" (id 1) (at 142.24 144.78 90))
     (property "Footprint" "libraries:SOT23" (id 2) (at 142.24 137.16 0)
       (effects (font (size 1.27 1.27)) (justify left bottom) hide)
@@
     (in_bom yes) (on_board yes) (fields_autoplaced)
     (property "Reference" "T4" (id 0) (at 127 142.24 90))
-    (property "Value" "" (id 1) (at 127 144.78 90))
+    (property "Value" "NTR4503" (id 1) (at 127 144.78 90))
     (property "Footprint" "libraries:SOT23" (id 2) (at 127 137.16 0)
       (effects (font (size 1.27 1.27)) (justify left bottom) hide)
@@
     (in_bom yes) (on_board yes) (fields_autoplaced)
     (property "Reference" "T5" (id 0) (at 142.24 119.38 90))
-    (property "Value" "" (id 1) (at 142.24 121.92 90))
+    (property "Value" "NTR4503" (id 1) (at 142.24 121.92 90))
     (property "Footprint" "libraries:SOT23" (id 2) (at 142.24 114.3 0)
       (effects (font (size 1.27 1.27)) (justify left bottom) hide)
@@
     (in_bom yes) (on_board yes) (fields_autoplaced)
     (property "Reference" "T7" (id 0) (at 157.48 142.24 90))
-    (property "Value" "" (id 1) (at 157.48 144.78 90))
+    (property "Value" "NTR4503" (id 1) (at 157.48 144.78 90))
     (property "Footprint" "libraries:SOT23" (id 2) (at 157.48 137.16 0)
       (effects (font (size 1.27 1.27)) (justify left bottom) hide)
@@
     (in_bom yes) (on_board yes) (fields_autoplaced)
     (property "Reference" "T2" (id 0) (at 111.76 142.24 90))
-    (property "Value" "" (id 1) (at 111.76 144.78 90))
+    (property "Value" "NTR4503" (id 1) (at 111.76 144.78 90))
     (property "Footprint" "libraries:SOT23" (id 2) (at 111.76 137.16 0)
       (effects (font (size 1.27 1.27)) (justify left bottom) hide)
@@
     (in_bom yes) (on_board yes) (fields_autoplaced)
     (property "Reference" "T3" (id 0) (at 127 119.38 90))
-    (property "Value" "" (id 1) (at 127 121.92 90))
+    (property "Value" "NTR4503" (id 1) (at 127 121.92 90))
     (property "Footprint" "libraries:SOT23" (id 2) (at 127 114.3 0)
       (effects (font (size 1.27 1.27)) (justify left bottom) hide)

Commit message: updates kroonsteentjes naar 2.54mm voor 7segment en buffer
Parts:
- J3: footprint libraries:TE_282841-8 -> (none)
Changed lines of the file:
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@@
       (effects (font (size 1.27 1.27)) (justify left))
     )
-    (property "Footprint" "libraries:TE_282841-8" (id 2) (at 176.53 121.92 0)
+    (property "Footprint" "" (id 2) (at 176.53 121.92 0)
       (effects (font (size 1.27 1.27)) hide)
     )
@@
     )
     (path "/1842b158-5de9-40ef-b815-cc6428c97c75"
-      (reference "J3") (unit 1) (value "R pinnen RGB strips") (footprint "libraries:TE_282841-8")
+      (reference "J3") (unit 1) (value "R pinnen RGB strips") (footprint "libraries:TE_1546215-8")
     )
     (path "/8adcd312-ab4a-4413-b6a5-effc7c373c70"

Commit message: aanmaak mapje voor finale ontwerpen
Parts:
- J2: footprint libraries:TE_282841-2 -> (none)
- J3: footprint (none) -> libraries:TE_1546215-8
Changed lines of the file:
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@@
       (effects (font (size 1.27 1.27)) (justify left))
     )
-    (property "Footprint" "" (id 2) (at 176.53 121.92 0)
+    (property "Footprint" "libraries:TE_1546215-8" (id 2) (at 176.53 121.92 0)
       (effects (font (size 1.27 1.27)) hide)
     )
@@
     (property "Reference" "J2" (id 0) (at 234.95 40.64 0))
     (property "Value" "12V DC" (id 1) (at 234.95 43.18 0))
-    (property "Footprint" "libraries:TE_282841-2" (id 2) (at 236.22 48.26 0)
+    (property "Footprint" "" (id 2) (at 236.22 48.26 0)
       (effects (font (size 1.27 1.27)) (justify left bottom) hide)
     )
@@
     )
     (path "/9d86002a-4404-4832-bfc8-aaaacfcac63c"
-      (reference "J2") (unit 1) (value "12V DC") (footprint "libraries:TE_282841-2")
+      (reference "J2") (unit 1) (value "12V DC") (footprint "libraries:TE_1546215-2")
     )
     (path "/1842b158-5de9-40ef-b815-cc6428c97c75"
