File: KiCad/fiets/poging 3/standaard.kicad_pcb (KiCad board)
At the start: 2 copper layers, 92.5 x 55.2 mm, 33 parts, among them J1 Conn_01x04_Female, J2 R pinnen RGB strips, J3 282837-4, J4 282841-2, J5 282841-2, SW1 ENABLE, SW2 BOOT, U1 ESP32-WROOM-32E_(16MB), U2 AMS1117, U3 BOB-12009

Commit message: aanpassingen kicad fiets
Parts:
- removed the R1 at (159.4, 44.7)
- moved R9 55.9 mm to (177.3, 67.4), turned to -90 degrees
- moved R8 55.8 mm to (173.3, 67.5), turned to -90 degrees
- moved U3 36.5 mm to (188.3, 71.1)
- moved C5 31.7 mm to (132.2, 34.9), turned to -90 degrees
- moved R1 30.9 mm to (153.7, 55.0), turned to -90 degrees
- moved CR3 23.2 mm to (161.0, 38.4)
- moved CR4 19.6 mm to (146.2, 35.8), turned to 0 degrees
- moved C8 18.5 mm to (171.3, 77.5), turned to 180 degrees
- moved J3 17.0 mm to (198.9, 34.6), turned to -90 degrees
- moved C6 16.7 mm to (177.3, 76.9)
- moved C9 14.7 mm to (171.1, 74.9), turned to 0 degrees
- moved CR1 14.7 mm to (160.8, 44.7)
- moved CR2 11.0 mm to (146.3, 39.1), turned to 0 degrees
- moved C1 9.90 mm to (146.5, 54.6)
- moved R3 9.64 mm to (146.3, 41.9)
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Connections:
- J2 pad 6: unconnected-(J2-Pad6) -> GND
Routing:
- net GND: track 426.2 -> 105.1 mm, vias 7 -> 4
- net Net-(C2-Pad1): track 0.00 -> 166.8 mm, vias 0 -> 1
- net Net-(C5-Pad2): track 57.0 -> 105.6 mm
- net Net-(C5-Pad1): track 0.00 -> 48.5 mm, vias 0 -> 2
- net Net-(R8-Pad2): track 0.00 -> 43.5 mm, vias 0 -> 1
- net Net-(J2-Pad5): track 62.9 -> 100.4 mm
- net Net-(C8-Pad2): track 49.7 -> 86.9 mm, vias 0 -> 1
- net Net-(C1-Pad2): track 67.5 -> 30.4 mm, vias 1 -> 0
- net +3V3: track 0.00 -> 35.3 mm, vias 0 -> 2
- net Net-(J3-Pad3): track 0.00 -> 22.3 mm
- net Net-(J2-Pad7): track 80.3 -> 98.2 mm
- net Net-(J1-Pad2): track 29.9 -> 16.9 mm
- net Net-(CR3-Pad1): track 24.4 -> 16.4 mm, vias 1 -> 0
- net Net-(R4-Pad1): track 9.90 -> 4.63 mm
- net Net-(J1-Pad3): track 11.4 -> 7.39 mm
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Other:
- board size 92.5 x 55.2 mm -> 92.5 x 57.5 mm
