File: KiCad/fiets/poging 3 (correct)/standaard.kicad_sch (KiCad schematic)
At the start: 32 parts, among them J1 Conn_01x04_Female, J2 R pinnen RGB strips, J3 282837-4, J4 282841-2, J5 282841-2, SW1 ENABLE, SW2 BOOT, U1 ESP32-WROOM-32E_(16MB), U2 AMS1117, U3 BOB-12009

Commit message: fiets hermaakt (2 versies level shifter)
Parts:
- J2: footprint libraries:TE_282841-8 -> (none)
- J3: footprint 282837-4:TE_282837-4 -> (none)
- J4, J5: footprint libraries:TE_282841-2 -> (none)
Connections:
- net +3V3: now also C2.1, C3.1, C4.1, C6.1, C7.1, J1.4 (Pin_4), U1.2 (3V3), U2.2 (VOUT), U2.4 (VOUT), U3.LV
Changed lines of the file:
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@@
   (junction (at 60.96 62.23) (diameter 0) (color 0 0 0 0)
+  )
+  (junction (at 111.76 54.61) (diameter 0) (color 0 0 0 0)
   )
   (junction (at 167.64 34.29) (diameter 0) (color 0 0 0 0)
@@
     (stroke (width 0) (type default) (color 0 0 0 0))
   )
-  (wire (pts (xy 111.76 50.8) (xy 111.76 57.15))
+  (wire (pts (xy 111.76 50.8) (xy 111.76 54.61))
     (stroke (width 0) (type default) (color 0 0 0 0))
   )
@@
     (stroke (width 0) (type default) (color 0 0 0 0))
   )
+  (wire (pts (xy 137.16 50.8) (xy 149.86 50.8))
+    (stroke (width 0) (type default) (color 0 0 0 0))
+  )
   (wire (pts (xy 172.72 88.9) (xy 172.72 93.98))
     (stroke (width 0) (type default) (color 0 0 0 0))
@@
     (stroke (width 0) (type default) (color 0 0 0 0))
   )
+  (wire (pts (xy 110.49 54.61) (xy 111.76 54.61))
+    (stroke (width 0) (type default) (color 0 0 0 0))
+  )
+  (wire (pts (xy 111.76 54.61) (xy 111.76 57.15))
+    (stroke (width 0) (type default) (color 0 0 0 0))
+  )
   (wire (pts (xy 177.8 76.2) (xy 177.8 99.06))
     (stroke (width 0) (type default) (color 0 0 0 0))
@@
   )
   (wire (pts (xy 111.76 115.57) (xy 137.16 115.57))
-    (stroke (width 0) (type default) (color 0 0 0 0))
-  )
-  (wire (pts (xy 137.16 50.8) (xy 149.86 50.8))
     (stroke (width 0) (type default) (color 0 0 0 0))
   )
@@
   (text "+" (at 209.55 54.61 0)
     (effects (font (size 1.27 1.27)) (justify left bottom))
+  )
+  (symbol (lib_id "power:+3V3") (at 110.49 54.61 0) (unit 1)
+    (in_bom yes) (on_board yes)
+    (property "Reference" "#PWR0108" (id 0) (at 110.49 58.42 0)
+      (effects (font (size 1.27 1.27)) hide)
+    )
+    (property "Value" "+3V3" (id 1) (at 110.49 50.8 0))
+    (property "Footprint" "" (id 2) (at 110.49 54.61 0)
+      (effects (font (size 1.27 1.27)) hide)
+    )
+    (property "Datasheet" "" (id 3) (at 110.49 54.61 0)
+      (effects (font (size 1.27 1.27)) hide)
+    )
+    (pin "1")
   )
   (symbol (lib_id "Device:R") (at 115.57 85.09 90) (unit 1)
@@
       (effects (font (size 1.27 1.27)) (justify right))
     )
-    (property "Footprint" "libraries:TE_282841-2" (id 2) (at 152.4 66.04 0)
+    (property "Footprint" "" (id 2) (at 152.4 66.04 0)
       (effects (font (size 1.27 1.27)) (justify left bottom) hide)
     )
@@
       (effects (font (size 1.27 1.27)) (justify left))
     )
-    (property "Footprint" "282837-4:TE_282837-4" (id 2) (at 170.18 134.62 0)
+    (property "Footprint" "" (id 2) (at 170.18 134.62 0)
       (effects (font (size 1.27 1.27)) (justify left bottom) hide)
     )
@@
       (effects (font (size 1.27 1.27)) (justify right))
     )
-    (property "Footprint" "libraries:TE_282841-2" (id 2) (at 217.17 46.99 0)
+    (property "Footprint" "" (id 2) (at 217.17 46.99 0)
       (effects (font (size 1.27 1.27)) (justify left bottom) hide)
     )
@@
       (effects (font (size 1.27 1.27)) (justify left))
     )
-    (property "Footprint" "libraries:TE_282841-8" (id 2) (at 135.89 99.06 0)
+    (property "Footprint" "" (id 2) (at 135.89 99.06 0)
       (effects (font (size 1.27 1.27)) hide)
     )
@@
       (reference "#PWR0107") (unit 1) (value "+3V3") (footprint "")
     )
+    (path "/0319edc6-d20a-4058-910f-ebe4e5090068"
+      (reference "#PWR0108") (unit 1) (value "+3V3") (footprint "")
+    )
     (path "/590c7ce0-b9ae-45c9-adef-24833a8dc22d"
       (reference "C1") (unit 1) (value "1u") (footprint "Capacitor_SMD:C_0805_2012Metric_Pad1.18x1.45mm_HandSolder")
@@
     )
     (path "/cb83f3f2-b69b-4c0c-ae2e-66da890134f0"
-      (reference "J2") (unit 1) (value "R pinnen RGB strips") (footprint "libraries:TE_282841-8")
+      (reference "J2") (unit 1) (value "R pinnen RGB strips") (footprint "libraries:TE_1546215-8")
     )
     (path "/571531e1-2047-40e6-a979-cd00b41e9e0f"
-      (reference "J3") (unit 1) (value "282837-4") (footprint "282837-4:TE_282837-4")
+      (reference "J3") (unit 1) (value "282837-4") (footprint "libraries:TE_1546215-4")
     )
     (path "/55ff87b6-13ce-4177-b1d3-b3df58f45f4c"
-      (reference "J4") (unit 1) (value "282841-2") (footprint "libraries:TE_282841-2")
+      (reference "J4") (unit 1) (value "282841-2") (footprint "libraries:TE_1546215-2")
     )
     (path "/b3e8ee36-4889-465f-962b-e5f603e0da07"
-      (reference "J5") (unit 1) (value "282841-2") (footprint "libraries:TE_282841-2")
+      (reference "J5") (unit 1) (value "282841-2") (footprint "libraries:TE_1546215-2")
     )
     (path "/6941509e-d537-4d22-8220-b842711d1953"
