File: KiCad/PCB Ontwerpen/Fiets - zelfgemaakte level shifter/standaard.kicad_pcb (KiCad board)
At the start: 2 copper layers, 80.6 x 56.7 mm, 37 parts, among them J1 Conn_01x04_Female, J2 R pinnen RGB strips, J3 282837-4, J4 282841-2, J5 282841-2, Q1 2N7002, Q2 2N7002, SW1 ENABLE, SW2 BOOT, U1 ESP32-WROOM-32E_(16MB)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

Commit message: laatste aanpassingen aan pcb ontwerpen
Routing:
- net GND: track 89.4 -> 82.9 mm
Changed lines of the file:
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@@
   (via (at 187.709 39.6308) (size 2) (drill 1) (layers "F.Cu" "B.Cu") (free) (net 1))
   (via (at 126.1872 75.692) (size 2) (drill 1) (layers "F.Cu" "B.Cu") (free) (net 1))
-  (segment (start 161.5588 51.5632) (end 161.5588 58.0632) (width 0.7) (layer "B.Cu") (net 1))
   (segment (start 157.5042 51.5632) (end 163.93615 45.13125) (width 0.7) (layer "F.Cu") (net 2))
   (segment (start 148.6756 55.7116) (end 147.574 54.61) (width 0.7) (layer "F.Cu") (net 2))
