File: KiCad/Buffer/hernieuwdeBuffer_beide_groundplane/hernieuwdeBuffer_beide_groundplane.kicad_pcb (KiCad board)
At the start: 2 copper layers, 111.8 x 77.5 mm, 44 parts, among them J1 Conn_01x04_Female, J2 DCJ200-10-A-XX-X_REVA, J3 Rood, J4 Groen, J5 Oranje1, J6 Oranje2, SW1 ENABLE, SW2 BOOT, T1 signaal oranje, T10 o3r, T11 o4r, T12 o5r, T13 06r, T14 r1, T15 r2, T16 r3, T17 r4, T18 r5, T19 g1, T2 o1g, T20 g2, T21 g3, T22 g4, T23 g5, T3 o2g, T4 o3g, T5 o4g, T6 o5g, T7 06g, T8 o1r, T9 o2r, U1 ESP32-WROOM-32E_(16MB), U2 AMS1117

Commit message: cut-outs groundplanes onder antenne
enkel voor 7 segments en buffer
Routing:
- net GND: vias 0 -> 4
Changed lines of the file:
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@@
   (segment (start 121.3625 86.8875) (end 121.35 86.9) (width 0.8) (layer "F.Cu") (net 1))
   (segment (start 174.3 93.45) (end 174.3 96.2) (width 0.8) (layer "F.Cu") (net 1))
+  (via (at 187.475 69.075) (size 2) (drill 1) (layers "F.Cu" "B.Cu") (free) (net 1))
+  (via (at 109.675 71.2) (size 2) (drill 1) (layers "F.Cu" "B.Cu") (free) (net 1))
+  (via (at 104.475 134.625) (size 2) (drill 1) (layers "F.Cu" "B.Cu") (free) (net 1))
+  (via (at 187.525 128.075) (size 2) (drill 1) (layers "F.Cu" "B.Cu") (free) (net 1))
   (segment (start 184.0975 88.5) (end 185.1375 89.54) (width 0.8) (layer "F.Cu") (net 2))
   (segment (start 171.1 88.5) (end 184.0975 88.5) (width 0.8) (layer "F.Cu") (net 2))
@@
       )
     )
+    (polygon
+      (pts
+        (xy 141.275 85.45)
+        (xy 141.275 93.3)
+        (xy 161.3 93.3)
+        (xy 161.3 85.45)
+      )
+    )

Commit message: updates kroonsteentjes naar 2.54mm voor 7segment en buffer
Parts:
- J3, J4: footprint libraries:TE_282841-5 -> libraries:TE_1546215-5
- J5, J6: footprint libraries:TE_282841-6 -> libraries:TE_1546215-6
- moved J5 13.8 mm to (99.3, 98.5)
- moved J4 6.61 mm to (167.1, 128.0)
- moved J6 1.80 mm to (99.3, 118.3)
- moved T10 1.10 mm to (119.5, 109.1)
Connections:
- C7 pad 2: unconnected-(C7-Pad2) -> Net-(C7-Pad2)
- C8 pad 1: unconnected-(C7-Pad2) -> Net-(C7-Pad2)
- J2 pad 1: unconnected-(J2-Pad1) -> Net-(PS1-Pad1b)
- PS1 pad 1b: unconnected-(J2-Pad1) -> Net-(PS1-Pad1b)
- PS1 pad 3b: unconnected-(C7-Pad2) -> Net-(C7-Pad2)
- U2 pad 3: unconnected-(C7-Pad2) -> Net-(C7-Pad2)
Routing:
- net Net-(C7-Pad2): track 0.00 -> 54.1 mm, vias 0 -> 1
- net unconnected-(C7-Pad2): track 47.6 -> 0.00 mm, vias 1 -> 0
- net unconnected-(J2-Pad1): track 15.3 -> 0.00 mm
- net Net-(PS1-Pad1b): track 0.00 -> 15.3 mm
- net g5: track 9.94 -> 19.6 mm
- net o1r: track 27.7 -> 18.9 mm
- net o1g: track 34.8 -> 27.2 mm
- net o2r: track 27.1 -> 19.5 mm
- net o2g: track 34.1 -> 26.6 mm
- net o3g: track 32.8 -> 27.1 mm
- net r1: track 16.4 -> 21.5 mm
- net g4: track 12.4 -> 8.23 mm
- net o3r: track 24.3 -> 20.9 mm
- net o4r: track 21.4 -> 18.3 mm
- net g3: track 14.8 -> 12.0 mm
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
Commit message: kopiëren van juiste pcb naar mapje over buffer
Other:
- board text added: "13"
- board text added: "16"
- board text added: "17"
- board text added: "18"
- board text added: "19"
- board text added: "21"
- board text added: "22"
- board text added: "23"
- board text added: "4"
- board text added: "5"
- board text added: "BUFFER"
- board text added: "GROEN"
- board text added: "ORANJE"
- board text added: "ROOD"
- board text added: "g 12 r"
- board text added: "g 14 r"
- board text added: "g 25 r"
- board text added: "g 26 r"
- board text added: "g 27 r"
- board text added: "g 33 r"
Changed lines of the file:
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@@
       (effects (font (size 1 1) (thickness 0.15)))
     )
-    (fp_text user "ANTENNA" (at -6 -9) (layer "F.Fab")
+    (fp_text user "ANTENNA" (at -0.3125 -9.45) (layer "F.Fab")
       (effects (font (size 1.4 1.4) (thickness 0.15)))
     )
@@
   )
   (gr_rect (start 86.36 62.23) (end 198.12 139.7) (layer "Edge.Cuts") (width 0.1) (fill none))
+  (gr_text "ROOD" (at 187.2 108) (layer "F.Cu")
+    (effects (font (size 0.5 0.5) (thickness 0.125)))
+  )
+  (gr_text "17" (at 169.5 133) (layer "F.Cu")
+    (effects (font (size 0.5 0.5) (thickness 0.125)))
+  )
+  (gr_text "16" (at 167 133) (layer "F.Cu")
+    (effects (font (size 0.5 0.5) (thickness 0.125)))
+  )
+  (gr_text "g 33 r" (at 94.9 93.3 270) (layer "F.Cu")
+    (effects (font (size 0.5 0.5) (thickness 0.125)))
+  )
+  (gr_text "22" (at 190 97.5 90) (layer "F.Cu")
+    (effects (font (size 0.5 0.5) (thickness 0.125)))
+  )
+  (gr_text "g 25 r" (at 94.9 98.4 270) (layer "F.Cu")
+    (effects (font (size 0.5 0.5) (thickness 0.125)))
+  )
+  (gr_text "21" (at 190 100 90) (layer "F.Cu")
+    (effects (font (size 0.5 0.5) (thickness 0.125)))
+  )
+  (gr_text "g 14 r" (at 95 118 270) (layer "F.Cu")
+    (effects (font (size 0.5 0.5) (thickness 0.125)))
+  )
+  (gr_text "4" (at 164.5 133) (layer "F.Cu")
+    (effects (font (size 0.5 0.5) (thickness 0.125)))
+  )
+  (gr_text "g 26 r" (at 94.9 103.4 270) (layer "F.Cu")
+    (effects (font (size 0.5 0.5) (thickness 0.125)))
+  )
+  (gr_text "13" (at 162 133) (layer "F.Cu")
+    (effects (font (size 0.5 0.5) (thickness 0.125)))
+  )
+  (gr_text "5" (at 172 133) (layer "F.Cu")
+    (effects (font (size 0.5 0.5) (thickness 0.125)))
+  )
+  (gr_text "18" (at 190 105 90) (layer "F.Cu")
+    (effects (font (size 0.5 0.5) (thickness 0.125)))
+  )
+  (gr_text "ORANJE" (at 99.3 108.4) (layer "F.Cu")
+    (effects (font (size 0.5 0.5) (thickness 0.125)))
+  )
+  (gr_text "BUFFER" (at 107.5 69) (layer "F.Cu")
+    (effects (font (size 1.5 1.5) (thickness 0.375)))
+  )
+  (gr_text "g 12 r" (at 95 123 270) (layer "F.Cu")
+    (effects (font (size 0.5 0.5) (thickness 0.125)))
+  )
+  (gr_text "GROEN" (at 157.3 130.6) (layer "F.Cu")
+    (effects (font (size 0.5 0.5) (thickness 0.125)))
+  )
+  (gr_text "g 27 r" (at 95 113 270) (layer "F.Cu")
+    (effects (font (size 0.5 0.5) (thickness 0.125)))
+  )
+  (gr_text "19" (at 190 102.5 90) (layer "F.Cu")
+    (effects (font (size 0.5 0.5) (thickness 0.125)))
+  )
+  (gr_text "23" (at 190 95 90) (layer "F.Cu")
+    (effects (font (size 0.5 0.5) (thickness 0.125)))
+  )
   (target plus (at 91.44 135.89) (size 5) (width 0.1) (layer "Edge.Cuts"))
   (target plus (at 194.31 134.62) (size 5) (width 0.1) (layer "Edge.Cuts"))
@@
     (polygon
       (pts
-        (xy 198.12 137.16)
-        (xy 86.36 137.16)
-        (xy 86.36 59.69)
-        (xy 198.12 59.69)
+        (xy 198.12 139.76)
+        (xy 86.36 139.76)
+        (xy 86.36 62.19)
+        (xy 198.12 62.19)
       )
     )
