File: KiCad/PCB Ontwerpen/7 segment/7segments_beide_groundplane.kicad_sch (KiCad schematic)
At the start: 25 parts, among them J1 Conn_01x04_Female, J2 12V DC, J3 R pinnen RGB strips, SW1 ENABLE, SW2 BOOT, T1 NTR4503, T2 NTR4503, T3 NTR4503, T4 NTR4503, T5 NTR4503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

Commit message: aanpassing 7 segment naar dc jack
Parts:
- removed J2: 12V DC, symbol 282841-2:282841-2
- added J2: DCJ200-10-A-XX-X_REVA, libraries:GCT_DCJ200-10-A-XX-X_REVA, symbol DCJ200-10-A-XX-X_REVA:DCJ200-10-A-XX-X_REVA
Connections:
- net 12V: now also J2.1
- net GND: now also J2.2, J2.3
Changed lines of the file:
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@@
   (junction (at 132.08 81.28) (diameter 0) (color 0 0 0 0)
+  )
+  (junction (at 231.14 48.26) (diameter 0) (color 0 0 0 0)
   )
   (junction (at 116.84 55.88) (diameter 0) (color 0 0 0 0)
@@
   (no_connect (at 101.6 91.44))
   (no_connect (at 101.6 86.36))
+  (wire (pts (xy 231.14 45.72) (xy 231.14 48.26))
+    (stroke (width 0) (type default) (color 0 0 0 0))
+  )
   (wire (pts (xy 158.75 129.54) (xy 158.75 106.68))
     (stroke (width 0) (type default) (color 0 0 0 0))
@@
     (stroke (width 0) (type default) (color 0 0 0 0))
   )
+  (wire (pts (xy 231.14 48.26) (xy 231.14 50.8))
+    (stroke (width 0) (type default) (color 0 0 0 0))
+  )
   (wire (pts (xy 33.02 96.52) (xy 33.02 99.06))
     (stroke (width 0) (type default) (color 0 0 0 0))
@@
     (stroke (width 0) (type default) (color 0 0 0 0))
   )
-  (wire (pts (xy 215.9 55.88) (xy 217.17 55.88))
+  (wire (pts (xy 215.9 55.88) (xy 231.14 55.88))
     (stroke (width 0) (type default) (color 0 0 0 0))
   )
@@
     (stroke (width 0) (type default) (color 0 0 0 0))
   )
+  (wire (pts (xy 222.25 48.26) (xy 231.14 48.26))
+    (stroke (width 0) (type default) (color 0 0 0 0))
+  )
   (wire (pts (xy 55.88 114.3) (xy 60.96 114.3))
     (stroke (width 0) (type default) (color 0 0 0 0))
@@
     (stroke (width 0) (type default) (color 0 0 0 0))
   )
-  (wire (pts (xy 217.17 50.8) (xy 226.06 50.8))
-    (stroke (width 0) (type default) (color 0 0 0 0))
-  )
   (wire (pts (xy 101.6 132.08) (xy 111.76 132.08))
     (stroke (width 0) (type default) (color 0 0 0 0))
@@
     (stroke (width 0) (type default) (color 0 0 0 0))
   )
-  (wire (pts (xy 222.25 48.26) (xy 226.06 48.26))
-    (stroke (width 0) (type default) (color 0 0 0 0))
-  )
   (wire (pts (xy 146.05 39.37) (xy 146.05 48.26))
     (stroke (width 0) (type default) (color 0 0 0 0))
@@
   )
   (wire (pts (xy 142.24 124.46) (xy 142.24 134.62))
-    (stroke (width 0) (type default) (color 0 0 0 0))
-  )
-  (wire (pts (xy 217.17 55.88) (xy 217.17 50.8))
     (stroke (width 0) (type default) (color 0 0 0 0))
   )
@@
     )
   )
-  (global_label "12V" (shape input) (at 222.25 50.8 270) (fields_autoplaced)
+  (global_label "12V" (shape input) (at 222.25 55.88 270) (fields_autoplaced)
     (effects (font (size 1.27 1.27)) (justify right))
-    (property "Intersheet References" "${INTERSHEET_REFS}" (id 0) (at 222.1706 56.7207 90)
+    (property "Intersheet References" "${INTERSHEET_REFS}" (id 0) (at 222.1706 61.8007 90)
       (effects (font (size 1.27 1.27)) (justify right) hide)
     )
@@
     (pin "3")
   )
-  (symbol (lib_id "282841-2:282841-2") (at 236.22 48.26 0) (mirror x) (unit 1)
-    (in_bom yes) (on_board yes) (fields_autoplaced)
-    (property "Reference" "J2" (id 0) (at 234.95 40.64 0))
-    (property "Value" "12V DC" (id 1) (at 234.95 43.18 0))
-    (property "Footprint" "" (id 2) (at 236.22 48.26 0)
-      (effects (font (size 1.27 1.27)) (justify left bottom) hide)
-    )
-    (property "Datasheet" "" (id 3) (at 236.22 48.26 0)
-      (effects (font (size 1.27 1.27)) (justify left bottom) hide)
-    )
-    (property "Comment" "282841-2" (id 4) (at 236.22 48.26 0)
-      (effects (font (size 1.27 1.27)) (justify left bottom) hide)
-    )
-    (property "EU_RoHS_Compliance" "Compliant with Exemptions" (id 5) (at 236.22 48.26 0)
-      (effects (font (size 1.27 1.27)) (justify left bottom) hide)
-    )
-    (pin "1")
-    (pin "2")
-  )
   (symbol (lib_id "AMS1117:AMS1117") (at 165.1 53.34 180) (unit 1)
     (in_bom yes) (on_board yes) (fields_autoplaced)
@@
     (pin "1")
   )
+  (symbol (lib_id "DCJ200-10-A-XX-X_REVA:DCJ200-10-A-XX-X_REVA") (at 238.76 50.8 180) (unit 1)
+    (in_bom yes) (on_board yes) (fields_autoplaced)
+    (property "Reference" "J2" (id 0) (at 245.11 50.7999 0)
+      (effects (font (size 1.27 1.27)) (justify right))
+    )
+    (property "Value" "DCJ200-10-A-XX-X_REVA" (id 1) (at 245.11 53.3399 0)
+      (effects (font (size 1.27 1.27)) (justify right))
+    )
+    (property "Footprint" "libraries:GCT_DCJ200-10-A-XX-X_REVA" (id 2) (at 238.76 50.8 0)
+      (effects (font (size 1.27 1.27)) (justify left bottom) hide)
+    )
+    (property "Datasheet" "" (id 3) (at 238.76 50.8 0)
+      (effects (font (size 1.27 1.27)) (justify left bottom) hide)
+    )
+    (property "MANUFACTURER" "GCT" (id 4) (at 238.76 50.8 0)
+      (effects (font (size 1.27 1.27)) (justify left bottom) hide)
+    )
+    (pin "1")
+    (pin "2")
+    (pin "3")
+  )
   (symbol (lib_id "BC848:BC848") (at 127 114.3 270) (unit 1)
     (in_bom yes) (on_board yes) (fields_autoplaced)
@@
       (reference "J1") (unit 1) (value "Conn_01x04_Female") (footprint "Connector_PinHeader_2.54mm:PinHeader_1x04_P2.54mm_Vertical")
     )
-    (path "/9d86002a-4404-4832-bfc8-aaaacfcac63c"
-      (reference "J2") (unit 1) (value "12V DC") (footprint "libraries:TE_1546215-2")
+    (path "/e174db42-2133-4bde-8bf0-5dfc27789f4d"
+      (reference "J2") (unit 1) (value "DCJ200-10-A-XX-X_REVA") (footprint "libraries:GCT_DCJ200-10-A-XX-X_REVA")
     )
     (path "/1842b158-5de9-40ef-b815-cc6428c97c75"
