File: KiCad/Kicad-versie Bert/Fiets - zelfgemaakte level shifter/Fiets - zelfgemaakte level shifter/standaard.kicad_pcb (KiCad board)
At the start: 2 copper layers, 72.8 x 40.4 mm, 36 parts, among them J1 Conn_01x04_Female, J4 282841-2, J5 282841-2, Q1 2N7002, Q2 2N7002, SW1 ENABLE, SW2 BOOT, U1 ESP32-WROOM-32E_(16MB), U2 AMS1117

Commit message: goed code toevoegen, fotos website, ...
Parts:
- turned R2 to 180 degrees
- renumbered RGB to J2, LCD to J3
Connections:
- C5 pad 1: Net-(C5-Pad1) -> Net-(CR2-Pad1)
- C5 pad 2: Net-(C5-Pad2) -> GND
- CR1 pad 2: Net-(C5-Pad1) -> GND
- CR2 pad 1: Net-(C5-Pad2) -> Net-(CR2-Pad1)
- CR3 pad 2: Net-(C5-Pad1) -> GND
- CR4 pad 1: Net-(C5-Pad2) -> Net-(CR2-Pad1)
- R2 pad 1: Net-(C5-Pad1) -> Net-(R2-Pad1)
- R2 pad 2: GND -> Net-(CR2-Pad1)
- R3 pad 2: Net-(C5-Pad2) -> Net-(R2-Pad1)
- U1 pad 6: Net-(C5-Pad2) -> Net-(R2-Pad1)
Routing:
- net Net-(CR2-Pad1): track 0.00 -> 59.2 mm, vias 0 -> 1
- net Net-(C5-Pad2): track 48.2 -> 0.00 mm
- net Net-(C5-Pad1): track 30.3 -> 0.00 mm
- net Net-(R2-Pad1): track 0.00 -> 11.5 mm
- net GND: track 5.94 -> 9.55 mm
