File: KiCad/Kicad-versie Bert/Fiets - zelfgemaakte level shifter/Fiets - zelfgemaakte level shifter/standaard.kicad_pcb (KiCad board)
At the start: 2 copper layers, 72.8 x 40.4 mm, 36 parts, among them J1 Conn_01x04_Female, J4 282841-2, J5 282841-2, Q1 2N7002, Q2 2N7002, SW1 ENABLE, SW2 BOOT, U1 ESP32-WROOM-32E_(16MB), U2 AMS1117

Commit message: aanpassingen aan eeschema en pcb fiets
spanningsdeler gewijzigd en condensator juist georiënteerd
Parts:
- R2: value 560 -> 120
- R3: value 120 -> 560
- moved C5 33.2 mm to (139.8, 66.2), turned to 90 degrees
- moved R3 4.03 mm to (158.4, 44.7), turned to 180 degrees
- moved R2 3.82 mm to (162.9, 43.2), turned to 180 degrees
- moved CR3 1.38 mm to (158.8, 38.9)
- renumbered RGB to J2, LCD to J3
Connections:
- C5 pad 2: Net-(C5-Pad2) -> GND
- CR1 pad 2: Net-(C5-Pad1) -> GND
- CR2 pad 1: Net-(C5-Pad2) -> Net-(C5-Pad1)
- CR3 pad 2: Net-(C5-Pad1) -> GND
- CR4 pad 1: Net-(C5-Pad2) -> Net-(C5-Pad1)
- R2 pad 1: Net-(C5-Pad1) -> GND
- R2 pad 2: GND -> Net-(R2-Pad2)
- R3 pad 1: GND -> Net-(R2-Pad2)
- R3 pad 2: Net-(C5-Pad2) -> Net-(C5-Pad1)
- U1 pad 6: Net-(C5-Pad2) -> Net-(R2-Pad2)
Routing:
- net Net-(C5-Pad2): track 48.2 -> 0.00 mm
- net Net-(R2-Pad2): track 0.00 -> 14.0 mm
- net Net-(C5-Pad1): track 30.3 -> 41.0 mm
- net Net-(CR3-Pad1): track 12.1 -> 10.9 mm
