File: KiCad/Kicad-versie Bert/Fiets - zelfgemaakte level shifter/Fiets - zelfgemaakte level shifter/standaard.kicad_sch (KiCad schematic)
At the start: 36 parts, among them J1 Conn_01x04_Female, Q1 2N7002, Q2 2N7002, SW1 ENABLE, SW2 BOOT, U2 AMS1117

Commit message: goed code toevoegen, fotos website, ...
Parts:
- J2: value (none) -> Conn_01x07_Male; footprint (none) -> Connector_PinHeader_2.54mm:PinHeader_1x07_P2.54mm_Vertical
- J3: value (none) -> 282837-4; footprint (none) -> Connector_PinHeader_2.54mm:PinHeader_1x04_P2.54mm_Vertical
- J4, J5: value (none) -> 282841-2; footprint (none) -> Connector_PinHeader_2.54mm:PinHeader_1x02_P2.54mm_Vertical
- U1: value (none) -> ESP32-WROOM-32E_(16MB); footprint (none) -> footprints:MODULE_ESP32-WROOM-32(8MB)
Connections:
- net GND: now also C5.2, CR1.2, CR3.2; no longer R2.2
- new net: R2.1, R3.2, U1.6 (IO34)
- new net: C5.1, CR2.1, CR4.1, R2.2
Other:
- moved on the sheet: C5, R2, R3
