File: KiCad/Kicad-versie Bert/Fiets - zelfgemaakte level shifter/Fiets - zelfgemaakte level shifter/standaard.kicad_sch (KiCad schematic)
At the start: 36 parts, among them J1 Conn_01x04_Female, Q1 2N7002, Q2 2N7002, SW1 ENABLE, SW2 BOOT, U2 AMS1117

Commit message: aanpassingen aan eeschema en pcb fiets
spanningsdeler gewijzigd en condensator juist georiënteerd
Parts:
- J2: value (none) -> Conn_01x07_Male; footprint (none) -> Connector_PinHeader_2.54mm:PinHeader_1x07_P2.54mm_Vertical
- J3: value (none) -> 282837-4; footprint (none) -> Connector_PinHeader_2.54mm:PinHeader_1x04_P2.54mm_Vertical
- J4, J5: value (none) -> 282841-2; footprint (none) -> Connector_PinHeader_2.54mm:PinHeader_1x02_P2.54mm_Vertical
- R2: value 560 -> 120
- R3: value 120 -> 560
- U1: value (none) -> ESP32-WROOM-32E_(16MB); footprint (none) -> footprints:MODULE_ESP32-WROOM-32(8MB)
Connections:
- net GND: now also C5.2, CR1.2, CR3.2, R2.1; no longer R2.2, R3.1
- net at CR2.1, CR4.1, R3.2: now also C5.1; no longer C5.2, U1.6 (IO34)
- new net: R2.2, R3.1, U1.6 (IO34)
Other:
- moved on the sheet: C5
Changed lines of the file:
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@@
   (junction (at 128.27 180.34) (diameter 0) (color 0 0 0 0)
   )
+  (junction (at 154.94 115.57) (diameter 0) (color 0 0 0 0)
+  )
+  (junction (at 60.96 67.31) (diameter 0) (color 0 0 0 0)
+  )
+  (junction (at 151.13 129.54) (diameter 0) (color 0 0 0 0)
+  )
+  (junction (at 111.76 57.15) (diameter 0) (color 0 0 0 0)
+  )
+  (junction (at 154.94 106.68) (diameter 0) (color 0 0 0 0)
+  )
+  (junction (at 40.64 67.31) (diameter 0) (color 0 0 0 0)
+  )
+  (junction (at 189.23 34.29) (diameter 0) (color 0 0 0 0)
+  )
+  (junction (at 158.75 76.2) (diameter 0) (color 0 0 0 0)
+  )
   (junction (at 168.91 106.68) (diameter 0) (color 0 0 0 0)
   )
-  (junction (at 60.96 67.31) (diameter 0) (color 0 0 0 0)
-  )
-  (junction (at 151.13 129.54) (diameter 0) (color 0 0 0 0)
-  )
-  (junction (at 111.76 57.15) (diameter 0) (color 0 0 0 0)
-  )
-  (junction (at 40.64 67.31) (diameter 0) (color 0 0 0 0)
-  )
-  (junction (at 181.61 106.68) (diameter 0) (color 0 0 0 0)
-  )
-  (junction (at 189.23 34.29) (diameter 0) (color 0 0 0 0)
-  )
-  (junction (at 158.75 76.2) (diameter 0) (color 0 0 0 0)
-  )
   (junction (at 189.23 43.18) (diameter 0) (color 0 0 0 0)
   )
@@
   )
   (junction (at 154.94 50.8) (diameter 0) (color 0 0 0 0)
-  )
-  (junction (at 157.48 115.57) (diameter 0) (color 0 0 0 0)
   )
   (junction (at 149.86 50.8) (diameter 0) (color 0 0 0 0)
@@
     (stroke (width 0) (type default) (color 0 0 0 0))
   )
-  (wire (pts (xy 168.91 106.68) (xy 168.91 115.57))
-    (stroke (width 0) (type default) (color 0 0 0 0))
-  )
   (wire (pts (xy 189.23 43.18) (xy 189.23 34.29))
     (stroke (width 0) (type default) (color 0 0 0 0))
   )
-  (wire (pts (xy 137.16 115.57) (xy 157.48 115.57))
+  (wire (pts (xy 137.16 115.57) (xy 154.94 115.57))
     (stroke (width 0) (type default) (color 0 0 0 0))
   )
@@
     (stroke (width 0) (type default) (color 0 0 0 0))
   )
+  (wire (pts (xy 168.91 106.68) (xy 168.91 121.92))
+    (stroke (width 0) (type default) (color 0 0 0 0))
+  )
   (wire (pts (xy 114.3 64.77) (xy 118.11 64.77))
     (stroke (width 0) (type default) (color 0 0 0 0))
@@
     (stroke (width 0) (type default) (color 0 0 0 0))
   )
+  (wire (pts (xy 154.94 106.68) (xy 154.94 115.57))
+    (stroke (width 0) (type default) (color 0 0 0 0))
+  )
   (wire (pts (xy 140.97 143.51) (xy 151.13 143.51))
     (stroke (width 0) (type default) (color 0 0 0 0))
@@
     (stroke (width 0) (type default) (color 0 0 0 0))
   )
-  (wire (pts (xy 181.61 106.68) (xy 181.61 121.92))
-    (stroke (width 0) (type default) (color 0 0 0 0))
-  )
   (wire (pts (xy 140.97 151.13) (xy 140.97 154.94))
     (stroke (width 0) (type default) (color 0 0 0 0))
@@
     (stroke (width 0) (type default) (color 0 0 0 0))
   )
-  (wire (pts (xy 157.48 115.57) (xy 168.91 115.57))
-    (stroke (width 0) (type default) (color 0 0 0 0))
-  )
   (wire (pts (xy 207.01 44.45) (xy 207.01 34.29))
     (stroke (width 0) (type default) (color 0 0 0 0))
@@
     (stroke (width 0) (type default) (color 0 0 0 0))
   )
-  (wire (pts (xy 57.15 121.92) (xy 181.61 121.92))
+  (wire (pts (xy 57.15 121.92) (xy 168.91 121.92))
     (stroke (width 0) (type default) (color 0 0 0 0))
   )
@@
   )
   (wire (pts (xy 60.96 62.23) (xy 67.31 62.23))
+    (stroke (width 0) (type default) (color 0 0 0 0))
+  )
+  (wire (pts (xy 154.94 115.57) (xy 157.48 115.57))
     (stroke (width 0) (type default) (color 0 0 0 0))
   )
@@
     (in_bom yes) (on_board yes)
     (property "Reference" "R2" (id 0) (at 161.29 101.6 90))
-    (property "Value" "560" (id 1) (at 161.29 104.14 90))
+    (property "Value" "120" (id 1) (at 161.29 104.14 90))
     (property "Footprint" "Resistor_SMD:R_0805_2012Metric_Pad1.20x1.40mm_HandSolder" (id 2) (at 161.29 106.68 0)
       (effects (font (size 1.27 1.27)) hide)
@@
       (effects (font (size 1.27 1.27)) (justify right))
     )
-    (property "Value" "" (id 1) (at 156.21 68.5799 90)
+    (property "Value" "282841-2" (id 1) (at 156.21 68.5799 90)
       (effects (font (size 1.27 1.27)) (justify right))
     )
-    (property "Footprint" "" (id 2) (at 152.4 66.04 0)
+    (property "Footprint" "Connector_PinHeader_2.54mm:PinHeader_1x02_P2.54mm_Vertical" (id 2) (at 152.4 66.04 0)
       (effects (font (size 1.27 1.27)) (justify left bottom) hide)
     )
@@
       (effects (font (size 1.27 1.27)) (justify left))
     )
-    (property "Value" "" (id 1) (at 176.53 134.6199 0)
-      (effects (font (size 1.27 1.27)) (justify left))
-    )
-    (property "Footprint" "" (id 2) (at 170.18 134.62 0)
+    (property "Value" "282837-4" (id 1) (at 176.53 134.6199 0)
+      (effects (font (size 1.27 1.27)) (justify left))
+    )
+    (property "Footprint" "Connector_PinHeader_2.54mm:PinHeader_1x04_P2.54mm_Vertical" (id 2) (at 170.18 134.62 0)
       (effects (font (size 1.27 1.27)) (justify left bottom) hide)
     )
@@
     (pin "2")
   )
-  (symbol (lib_id "Device:C_Polarized") (at 167.64 99.06 90) (mirror x) (unit 1)
-    (in_bom yes) (on_board yes)
-    (property "Reference" "C5" (id 0) (at 163.83 95.25 90))
-    (property "Value" "1000µ" (id 1) (at 168.91 95.25 90))
-    (property "Footprint" "Capacitor_THT:CP_Axial_L26.5mm_D20.0mm_P33.00mm_Horizontal" (id 2) (at 171.45 100.0252 0)
+  (symbol (lib_id "Device:C_Polarized") (at 167.64 99.06 270) (unit 1)
+    (in_bom yes) (on_board yes)
+    (property "Reference" "C5" (id 0) (at 171.45 95.25 90))
+    (property "Value" "1000µ" (id 1) (at 166.37 95.25 90))
+    (property "Footprint" "Capacitor_THT:CP_Axial_L26.5mm_D20.0mm_P33.00mm_Horizontal" (id 2) (at 163.83 100.0252 0)
       (effects (font (size 1.27 1.27)) hide)
     )
@@
       (effects (font (size 1.27 1.27)) (justify right))
     )
-    (property "Value" "" (id 1) (at 214.6301 50.8 90)
+    (property "Value" "282841-2" (id 1) (at 214.6301 50.8 90)
       (effects (font (size 1.27 1.27)) (justify right))
     )
-    (property "Footprint" "" (id 2) (at 217.17 46.99 0)
+    (property "Footprint" "Connector_PinHeader_2.54mm:PinHeader_1x02_P2.54mm_Vertical" (id 2) (at 217.17 46.99 0)
       (effects (font (size 1.27 1.27)) (justify left bottom) hide)
     )
@@
       (effects (font (size 1.27 1.27)) (justify right))
     )
-    (property "Value" "" (id 1) (at 135.3312 85.5222 0)
+    (property "Value" "Conn_01x07_Male" (id 1) (at 135.3312 85.5222 0)
       (effects (font (size 1.27 1.27)) (justify right))
     )
-    (property "Footprint" "" (id 2) (at 134.62 83.82 0)
+    (property "Footprint" "Connector_PinHeader_2.54mm:PinHeader_1x07_P2.54mm_Vertical" (id 2) (at 134.62 83.82 0)
       (effects (font (size 1.27 1.27)) hide)
     )
@@
     (in_bom yes) (on_board yes) (fields_autoplaced)
     (property "Reference" "U1" (id 0) (at 91.44 49.53 0))
-    (property "Value" "" (id 1) (at 91.44 52.07 0))
-    (property "Footprint" "" (id 2) (at 91.44 87.63 0)
+    (property "Value" "ESP32-WROOM-32E_(16MB)" (id 1) (at 91.44 52.07 0))
+    (property "Footprint" "footprints:MODULE_ESP32-WROOM-32(8MB)" (id 2) (at 91.44 87.63 0)
       (effects (font (size 1.27 1.27)) (justify left bottom) hide)
     )
@@
     (in_bom yes) (on_board yes)
     (property "Reference" "R3" (id 0) (at 175.26 101.6 90))
-    (property "Value" "120" (id 1) (at 175.26 104.14 90))
+    (property "Value" "560" (id 1) (at 175.26 104.14 90))
     (property "Footprint" "Resistor_SMD:R_0805_2012Metric_Pad1.20x1.40mm_HandSolder" (id 2) (at 175.26 106.68 0)
       (effects (font (size 1.27 1.27)) hide)
@@
     )
     (path "/0a364515-3e8d-4cd8-b418-7b3cee3740bc"
-      (reference "R2") (unit 1) (value "560") (footprint "Resistor_SMD:R_0805_2012Metric_Pad1.20x1.40mm_HandSolder")
+      (reference "R2") (unit 1) (value "120") (footprint "Resistor_SMD:R_0805_2012Metric_Pad1.20x1.40mm_HandSolder")
     )
     (path "/eeddac2a-5615-4b3b-a588-63b1af357dc6"
-      (reference "R3") (unit 1) (value "120") (footprint "Resistor_SMD:R_0805_2012Metric_Pad1.20x1.40mm_HandSolder")
+      (reference "R3") (unit 1) (value "560") (footprint "Resistor_SMD:R_0805_2012Metric_Pad1.20x1.40mm_HandSolder")
     )
     (path "/792a81e8-1972-4846-9d2f-a360e85a3cf8"
